File: pcbs/Platinen/eagle/Input_v1.0.brd (EAGLE design)
At the start: 100 x 77.4 mm, 157 parts, among them IC1 74HC14D, IC2 74HC14D, IC3 74AC573D, IC5 MAX485CSA, Q2 LFSPXO072036, U1 ATMEGA328P-AU-TQFP32, X1 SPT2.5/2-H-5.0, X2 SPT2.5/2-H-5.0, X3 SPT2.5/2-H-5.0, X4 SPT2.5/2-H-5.0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

Commit message: Bigger update 14.06.21
updated PCB files
updated documentation
updated RS485 protocol
updated firmwares
Parts:
- added R52, R53, R54, R55, R56, R57, R58: 10k, rcl:R0805
- R51: value (none) -> 10k; device resistor-bourns:4816P -> rcl:R0805
- X1, X2, X3, X4, X5: value SPT2.5/2-H-5.0 -> TBL009-500-02GY-2GY; device con-phoenix-500:SPT2 -> con-phoenix-500:TBL009-500-02GY-2GY
- moved R51 4.07 mm to (87.0, 37.1), turned to 270 degrees
- moved X1 2.71 mm to (11.4, 66.7)
- moved X2 2.71 mm to (21.6, 66.7)
- moved X3 2.71 mm to (44.5, 66.7)
- moved X4 2.71 mm to (54.6, 66.7)
- moved X5 2.71 mm to (33.0, 66.7)
Connections:
- net +5V: now also R51.2, R52.2, R53.2, R54.2, R55.2, R56.2, R57.2, R58.2; no longer R51.10, R51.11, R51.12, R51.13, R51.14, R51.15, R51.16, R51.9
- net D0: now also R52.1; no longer R51.1
- net D1: now also R51.1; no longer R51.2
- net D2: now also R53.1; no longer R51.3
- net D3: now also R54.1; no longer R51.4
- net D4: now also R55.1; no longer R51.5
- net D5: now also R56.1; no longer R51.6
- net D6: now also R57.1; no longer R51.7
- net D7: now also R58.1; no longer R51.8
- net GND1: now also X5.1.1, X5.1.2; no longer X5.2.1, X5.2.2
- net GND2: now also X5.2.1, X5.2.2; no longer X5.1.1, X5.1.2
- net N$15: now also X1.2.1, X1.2.2; no longer X1.1.1, X1.1.2
- net N$24: now also X2.1.1, X2.1.2; no longer X2.2.1, X2.2.2
- net N$33: now also X2.2.1, X2.2.2; no longer X2.1.1, X2.1.2
- net N$42: now also X3.1.1, X3.1.2; no longer X3.2.1, X3.2.2
- net N$51: now also X3.2.1, X3.2.2; no longer X3.1.1, X3.1.2
- net N$60: now also X4.1.1, X4.1.2; no longer X4.2.1, X4.2.2
- net N$69: now also X4.2.1, X4.2.2; no longer X4.1.1, X4.1.2
- net N$9: now also X1.1.1, X1.1.2; no longer X1.2.1, X1.2.2
- net RXD: now also IC5.1; no longer IC5.4
- net TXD: now also IC5.4; no longer IC5.1
Routing:
- net +5V: track 81.8 -> 110.6 mm
- net GND2: track 8.20 -> 0.00 mm
- net GND1: track 8.20 -> 0.00 mm
- net D2: track 105.7 -> 111.8 mm
- net D4: track 100.0 -> 106.0 mm
- net D0: track 104.4 -> 110.4 mm
- net D6: track 95.8 -> 101.8 mm
- net RXD: track 18.3 -> 14.5 mm
- net TXD: track 15.3 -> 18.4 mm
- net D7: track 87.6 -> 89.5 mm
- net D5: track 93.2 -> 95.1 mm
- net D3: track 97.1 -> 99.0 mm
- net D1: track 97.3 -> 99.2 mm
- net N$33: track 13.0 -> 12.4 mm
- net N$15: track 13.0 -> 12.4 mm
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Other:
- board text added: "SynPLC DI8-2 V1.0 05.07.20 Marco Müller"
- board text removed: "MicroSPS DI8-2 V1.0 05.07.20 Marco Müller"
