File: pcbs/Platinen/eagle/Input_v1.0.sch (EAGLE design)
At the start: 157 parts, among them IC1 74HC14D, IC2 74HC14D, IC3 74AC573D, IC5 MAX485CSA, Q2 LFSPXO072036, U1 ATMEGA328P-AU-TQFP32, X1 SPT2.5/2-H-5.0, X2 SPT2.5/2-H-5.0, X3 SPT2.5/2-H-5.0, X4 SPT2.5/2-H-5.0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

Commit message: Bigger update 14.06.21
updated PCB files
updated documentation
updated RS485 protocol
updated firmwares
Parts:
- added R52, R53, R54, R55, R56, R57, R58: 10k, rcl:R-EU_R0805
- R51: value (none) -> 10k; device resistor-bourns:4816P-T01 -> rcl:R-EU_R0805
- X1, X2, X3, X4, X5: value SPT2.5/2-H-5.0 -> TBL009-500-02GY-2GY; device con-phoenix-500:SPT2.5/2-H-5.0 -> con-phoenix-500:TBL009-500-02GY-2GY
Connections:
- net +5V: now also R51.2, R52.2, R53.2, R54.2, R55.2, R56.2, R57.2, R58.2; no longer R51.10, R51.11, R51.12, R51.13, R51.14, R51.15, R51.16, R51.9
- net D0: now also R52.1; no longer R51.1
- net D1: now also R51.1; no longer R51.2
- net D2: now also R53.1; no longer R51.3
- net D3: now also R54.1; no longer R51.4
- net D4: now also R55.1; no longer R51.5
- net D5: now also R56.1; no longer R51.6
- net D6: now also R57.1; no longer R51.7
- net D7: now also R58.1; no longer R51.8
- net GND1: now also X5.1; no longer X5.2
- net GND2: now also X5.2; no longer X5.1
- net N$15: now also X1.2; no longer X1.1
- net N$24: now also X2.1; no longer X2.2
- net N$33: now also X2.2; no longer X2.1
- net N$42: now also X3.1; no longer X3.2
- net N$51: now also X3.2; no longer X3.1
- net N$60: now also X4.1; no longer X4.2
- net N$69: now also X4.2; no longer X4.1
- net N$9: now also X1.1; no longer X1.2
- net RXD: now also IC5G$1.RO; no longer IC5G$1.DI
- net TXD: now also IC5G$1.DI; no longer IC5G$1.RO
