File: pcbs/Platinen/eagle/Output_v1.1.brd (EAGLE design)
At the start: 100 x 77.4 mm, 96 parts, among them IC1 74AC573D, IC2 74AC573D, IC3 74AC573D, IC4 ITS4880R, IC5 MAX485CSA, Q1 FQP27P06, Q2 LFSPXO072036, U1 ATMEGA328P-AU-TQFP32, X1 SPT2.5/2-H-5.0, X2 SPT2.5/2-H-5.0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

Commit message: Bigger update 14.06.21
updated PCB files
updated documentation
updated RS485 protocol
updated firmwares
Parts:
- added R28, R29, R30, R31, R32, R33, R34: 10k, rcl:R0805
- R11, R12, R13, R14, R15, R16, R17, R18: value (none) -> 1k5
- R27: value (none) -> 10k; device resistor-bourns:4816P -> rcl:R0805
- X1, X2, X3, X4, X5: value SPT2.5/2-H-5.0 -> TBL009-500-02GY-2GY; device con-phoenix-500:SPT2 -> con-phoenix-500:TBL009-500-02GY-2GY
- moved X2 21.1 mm to (50.2, 67.0)
- moved X1 21.1 mm to (40.0, 67.0)
- moved D1 20.6 mm to (78.4, 60.0)
- moved D3 20.6 mm to (68.3, 60.0)
- moved D8 20.6 mm to (42.9, 60.0)
- moved D6 20.6 mm to (53.0, 60.0)
- moved D5 20.0 mm to (58.1, 60.0)
- moved D2 20.0 mm to (73.3, 60.0)
- moved D4 20.0 mm to (63.2, 60.0)
- moved D7 20.0 mm to (47.9, 60.0)
- moved X3 19.9 mm to (60.3, 67.0)
- moved X4 19.9 mm to (70.5, 67.0)
- moved OK3 12.1 mm to (58.1, 46.7)
- moved OK4 10.8 mm to (46.7, 46.7)
- moved D19 10.2 mm to (61.3, 57.8)
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Connections:
- removed net N$28 (its old number): D1.C, D19.A, IC4.21, IC4.22, X4.1.1, X4.1.2
- new net N$27: D1.C, D19.A, IC4.21, IC4.22, X4.2.1, X4.2.2
- net +5V: now also R28.2, R29.2, R30.2, R31.2, R32.2, R33.2, R34.2; no longer R27.1, R27.3, R27.4, R27.5, R27.6, R27.7, R27.8
- net D0: now also R28.1; no longer R27.16
- net D1: now also R27.1; no longer R27.15
- net D2: now also R29.1; no longer R27.14
- net D3: now also R30.1; no longer R27.13
- net D4: now also R31.1; no longer R27.12
- net D5: now also R32.1; no longer R27.11
- net D6: now also R33.1; no longer R27.10
- net D7: now also R34.1; no longer R27.9
- net N$17: now also OK3.2; no longer OK4.2
- net N$18: now also OK3.4; no longer OK4.4
- net N$19: now also OK3.6; no longer OK4.6
- net N$20: now also OK3.8; no longer OK4.8
- net N$21: now also OK4.2; no longer OK3.2
- net N$22: now also OK4.4; no longer OK3.4
- net N$23: now also OK4.6; no longer OK3.6
- net N$24: now also OK4.8; no longer OK3.8
- net N$29: now also X4.1.1, X4.1.2; no longer X4.2.1, X4.2.2
- net N$30: now also X3.2.1, X3.2.2; no longer X3.1.1, X3.1.2
- net N$31: now also X3.1.1, X3.1.2; no longer X3.2.1, X3.2.2
- net N$32: now also X2.2.1, X2.2.2; no longer X2.1.1, X2.1.2
- net N$33: now also X2.1.1, X2.1.2; no longer X2.2.1, X2.2.2
- net N$34: now also X1.2.1, X1.2.2; no longer X1.1.1, X1.1.2
- net N$35: now also X1.1.1, X1.1.2; no longer X1.2.1, X1.2.2
- net RXD: now also IC5.1; no longer IC5.4
- net TXD: now also IC5.4; no longer IC5.1
Routing:
- net N$27: track 0.00 -> 93.0 mm, vias 0 -> 1
- net N$28 (its old number): track 58.9 -> 0.00 mm, vias 1 -> 0
- net N$29: track 50.6 -> 84.9 mm
- net N$30: track 43.3 -> 76.6 mm
- net N$31: track 37.8 -> 68.6 mm
- net +5V: track 64.5 -> 93.4 mm, vias 52 -> 48
- net N$33: track 76.6 -> 51.5 mm
- net N$34: track 68.6 -> 44.6 mm
- net N$32: track 82.7 -> 60.3 mm
- net N$35: track 60.1 -> 38.5 mm
- net N$38: track 47.6 -> 64.8 mm
- net N$37: track 52.0 -> 69.2 mm
- net N$39: track 47.5 -> 62.0 mm
- net N$36: track 58.9 -> 73.1 mm
- net +24V: track 35.7 -> 47.3 mm
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Other:
- board text added: "SynPLC DO8-1 V1.1 04.07.20 Marco Müller"
