File: pcbs/Platinen/eagle/Output_v1.1.sch (EAGLE design)
At the start: 96 parts, among them IC1 74AC573D, IC2 74AC573D, IC3 74AC573D, IC4 ITS4880R, IC5 MAX485CSA, Q1 FQP27P06, Q2 LFSPXO072036, U1 ATMEGA328P-AU-TQFP32, X1 SPT2.5/2-H-5.0, X2 SPT2.5/2-H-5.0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

Commit message: Bigger update 14.06.21
updated PCB files
updated documentation
updated RS485 protocol
updated firmwares
Parts:
- added R28, R29, R30, R31, R32, R33, R34: 10k, rcl:R-EU_R0805
- R11, R12, R13, R14, R15, R16, R17, R18: value (none) -> 1k5
- R27: value (none) -> 10k; device resistor-bourns:4816P-T01 -> rcl:R-EU_R0805
- X1, X2, X3, X4, X5: value SPT2.5/2-H-5.0 -> TBL009-500-02GY-2GY; device con-phoenix-500:SPT2.5/2-H-5.0 -> con-phoenix-500:TBL009-500-02GY-2GY
Connections:
- removed net N$28 (its old number): D1.C, D19.+, IC4.OUT8, IC4.OUT8@2, X4.1
- new net N$27: D1.C, D19.+, IC4.OUT8, IC4.OUT8@2, X4.2
- net +5V: now also R28.2, R29.2, R30.2, R31.2, R32.2, R33.2, R34.2; no longer R27.1, R27.3, R27.4, R27.5, R27.6, R27.7, R27.8
- net D0: now also R28.1; no longer R27.16
- net D1: now also R27.1; no longer R27.15
- net D2: now also R29.1; no longer R27.14
- net D3: now also R30.1; no longer R27.13
- net D4: now also R31.1; no longer R27.12
- net D5: now also R32.1; no longer R27.11
- net D6: now also R33.1; no longer R27.10
- net D7: now also R34.1; no longer R27.9
- net N$17: now also OK3A.C; no longer OK4A.C
- net N$18: now also OK3B.C; no longer OK4B.C
- net N$19: now also OK3C.C; no longer OK4C.C
- net N$20: now also OK3D.C; no longer OK4D.C
- net N$21: now also OK4A.C; no longer OK3A.C
- net N$22: now also OK4B.C; no longer OK3B.C
- net N$23: now also OK4C.C; no longer OK3C.C
- net N$24: now also OK4D.C; no longer OK3D.C
- net N$29: now also X4.1; no longer X4.2
- net N$30: now also X3.2; no longer X3.1
- net N$31: now also X3.1; no longer X3.2
- net N$32: now also X2.2; no longer X2.1
- net N$33: now also X2.1; no longer X2.2
- net N$34: now also X1.2; no longer X1.1
- net N$35: now also X1.1; no longer X1.2
- net RXD: now also IC5G$1.RO; no longer IC5G$1.DI
- net TXD: now also IC5G$1.DI; no longer IC5G$1.RO
Other:
- moved on the sheet: X1, X2, X3, X4
