File: pcbs/Platinen/kicad/AI_V1_revved/AI_V1.sch (KiCad schematic (older format))
At the start: 129 parts, among them J1 Conn_01x04, J10 TBL009-500-02GY-2GY, J11 TBL009-500-02GY-2GY, J2 Conn_01x02, J3 Conn_01x02, J4 Conn_02x03_Odd_Even, J5 Conn_02x05_Odd_Even, J6 Conn_02x05_Odd_Even, J7 TBL009-500-02GY-2GY, J8 TBL009-500-02GY-2GY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

Commit message: review AI V1 and AO V2
Parts:
- removed R44, R45, R46, R47: 1k, Resistor_SMD:R_0805_2012Metric_Pad1.20x1.40mm_HandSolder, symbol Device:R
- C22, C23, C24, C25, C32, C33, C34, C35: value 10p -> 10n
Connections:
- net SDA: now also U3.41 (PB5); no longer U3.43 (PB7)
- net at C38.2, U7.3 (+): now also FB1.2, R36.1
- net at C39.2, U8.3 (+): now also FB2.2, R38.1
- net at C40.2, U9.3 (+): now also FB3.2, R40.1
- net at C41.2, U10.3 (+): now also FB4.2, R42.1
Changed lines of the file:
@@
 	13550 1250 13750 1250
 Wire Wire Line
+	13750 1250 13750 850
+Wire Wire Line
 	13750 850  14200 850
 Connection ~ 13750 1250
@@
 P 12950 1800
 F 0 "C32" H 12835 1754 50  0000 R CNN
-F 1 "10p" H 12835 1845 50  0000 R CNN
+F 1 "10n" H 12835 1845 50  0000 R CNN
 F 2 "Capacitor_SMD:C_0805_2012Metric_Pad1.18x1.45mm_HandSolder" H 12988 1650 50  0001 C CNN
 F 3 "~" H 12950 1800 50  0001 C CNN
@@
 P 11300 1900
 F 0 "C22" H 11185 1854 50  0000 R CNN
-F 1 "10p" H 11185 1945 50  0000 R CNN
+F 1 "10n" H 11185 1945 50  0000 R CNN
 F 2 "Capacitor_SMD:C_0805_2012Metric_Pad1.18x1.45mm_HandSolder" H 11338 1750 50  0001 C CNN
 F 3 "~" H 11300 1900 50  0001 C CNN
@@
 	13550 2900 13750 2900
 Wire Wire Line
+	13750 2900 13750 2500
+Wire Wire Line
 	13750 2500 14200 2500
 Connection ~ 13750 2900
@@
 P 12950 3450
 F 0 "C33" H 12835 3404 50  0000 R CNN
-F 1 "10p" H 12835 3495 50  0000 R CNN
+F 1 "10n" H 12835 3495 50  0000 R CNN
 F 2 "Capacitor_SMD:C_0805_2012Metric_Pad1.18x1.45mm_HandSolder" H 12988 3300 50  0001 C CNN
 F 3 "~" H 12950 3450 50  0001 C CNN
@@
 P 11300 3550
 F 0 "C23" H 11185 3504 50  0000 R CNN
-F 1 "10p" H 11185 3595 50  0000 R CNN
+F 1 "10n" H 11185 3595 50  0000 R CNN
 F 2 "Capacitor_SMD:C_0805_2012Metric_Pad1.18x1.45mm_HandSolder" H 11338 3400 50  0001 C CNN
 F 3 "~" H 11300 3550 50  0001 C CNN
@@
 	13550 4550 13750 4550
 Wire Wire Line
+	13750 4550 13750 4150
+Wire Wire Line
 	13750 4150 14200 4150
 Connection ~ 13750 4550
@@
 P 12950 5100
 F 0 "C34" H 12835 5054 50  0000 R CNN
-F 1 "10p" H 12835 5145 50  0000 R CNN
+F 1 "10n" H 12835 5145 50  0000 R CNN
 F 2 "Capacitor_SMD:C_0805_2012Metric_Pad1.18x1.45mm_HandSolder" H 12988 4950 50  0001 C CNN
 F 3 "~" H 12950 5100 50  0001 C CNN
@@
 P 11300 5200
 F 0 "C24" H 11185 5154 50  0000 R CNN
-F 1 "10p" H 11185 5245 50  0000 R CNN
+F 1 "10n" H 11185 5245 50  0000 R CNN
 F 2 "Capacitor_SMD:C_0805_2012Metric_Pad1.18x1.45mm_HandSolder" H 11338 5050 50  0001 C CNN
 F 3 "~" H 11300 5200 50  0001 C CNN
@@
 	13550 6200 13750 6200
 Wire Wire Line
+	13750 6200 13750 5800
+Wire Wire Line
 	13750 5800 14200 5800
 Connection ~ 13750 6200
@@
 P 12950 6750
 F 0 "C35" H 12835 6704 50  0000 R CNN
-F 1 "10p" H 12835 6795 50  0000 R CNN
+F 1 "10n" H 12835 6795 50  0000 R CNN
 F 2 "Capacitor_SMD:C_0805_2012Metric_Pad1.18x1.45mm_HandSolder" H 12988 6600 50  0001 C CNN
 F 3 "~" H 12950 6750 50  0001 C CNN
@@
 P 11300 6850
 F 0 "C25" H 11185 6804 50  0000 R CNN
-F 1 "10p" H 11185 6895 50  0000 R CNN
+F 1 "10n" H 11185 6895 50  0000 R CNN
 F 2 "Capacitor_SMD:C_0805_2012Metric_Pad1.18x1.45mm_HandSolder" H 11338 6700 50  0001 C CNN
 F 3 "~" H 11300 6850 50  0001 C CNN
@@
 Wire Wire Line
 	4200 4550 4350 4550
-Text GLabel 2700 3850 0    50   Input ~ 0
+Text GLabel 2700 3650 0    50   Input ~ 0
 SDA
 Text GLabel 2700 3750 0    50   Input ~ 0
@@
 	2700 3750 2900 3750
 Wire Wire Line
-	2700 3850 2900 3850
+	2700 3650 2900 3650
 NoConn ~ 2900 3150
 NoConn ~ 2900 3250
 NoConn ~ 2900 3450
 NoConn ~ 2900 3550
+NoConn ~ 2900 3850
 NoConn ~ 2900 4450
 NoConn ~ 2900 4550
@@
 	13850 7000 13850 6750
 Connection ~ 13850 6750
-NoConn ~ 2900 3650
-Wire Wire Line
-	13750 1250 13750 1200
-Wire Wire Line
-	13750 2900 13750 2850
-Wire Wire Line
-	13750 4550 13750 4500
-Wire Wire Line
-	13750 6200 13750 6150
-$Comp
-L Device:R R47
-U 1 1 6118A9A4
-P 13750 6000
-F 0 "R47" H 13680 5954 50  0000 R CNN
-F 1 "1k" H 13680 6045 50  0000 R CNN
-F 2 "Resistor_SMD:R_0805_2012Metric_Pad1.20x1.40mm_HandSolder" V 13680 6000 50  0001 C CNN
-F 3 "~" H 13750 6000 50  0001 C CNN
-	1    13750 6000
-	-1   0    0    1
-$EndComp
-Wire Wire Line
-	13750 5850 13750 5800
-$Comp
-L Device:R R46
-U 1 1 6118C0C8
-P 13750 4350
-F 0 "R46" H 13680 4304 50  0000 R CNN
-F 1 "1k" H 13680 4395 50  0000 R CNN
-F 2 "Resistor_SMD:R_0805_2012Metric_Pad1.20x1.40mm_HandSolder" V 13680 4350 50  0001 C CNN
-F 3 "~" H 13750 4350 50  0001 C CNN
-	1    13750 4350
-	-1   0    0    1
-$EndComp
-Wire Wire Line
-	13750 4200 13750 4150
-$Comp
-L Device:R R45
-U 1 1 6118CCFA
-P 13750 2700
-F 0 "R45" H 13680 2654 50  0000 R CNN
-F 1 "1k" H 13680 2745 50  0000 R CNN
-F 2 "Resistor_SMD:R_0805_2012Metric_Pad1.20x1.40mm_HandSolder" V 13680 2700 50  0001 C CNN
-F 3 "~" H 13750 2700 50  0001 C CNN
-	1    13750 2700
-	-1   0    0    1
-$EndComp
-Wire Wire Line
-	13750 2550 13750 2500
-$Comp
-L Device:R R44
-U 1 1 6118D6EA
-P 13750 1050
-F 0 "R44" H 13680 1004 50  0000 R CNN
-F 1 "1k" H 13680 1095 50  0000 R CNN
-F 2 "Resistor_SMD:R_0805_2012Metric_Pad1.20x1.40mm_HandSolder" V 13680 1050 50  0001 C CNN
-F 3 "~" H 13750 1050 50  0001 C CNN
-	1    13750 1050
-	-1   0    0    1
-$EndComp
-Wire Wire Line
-	13750 900  13750 850
 $EndSCHEMATC
