File: pcbs/Platinen/kicad/AO_V2_revved/AO_V2.sch (KiCad schematic (older format))
At the start: 157 parts, among them J1 Conn_01x04, J10 Conn_01x02, J11 Conn_01x02, J2 Conn_02x03_Odd_Even, J3 Conn_02x05_Odd_Even, J4 Conn_02x05_Odd_Even, J5 TBL009-500-02GY-2GY, J6 TBL009-500-02GY-2GY, J7 TBL009-500-02GY-2GY, J8 TBL009-500-02GY-2GY, J9 TBL009-500-02GY-2GY, K1 G6K-2, K2 G6K-2, K3 G6K-2, K4 G6K-2, Q1 BC846, Q2 BC846, Q3 BC846, Q4 BC846, SW1 SW_DIP_x05, U1 SN65HVD232, U10 LM358, U11 LM358, U2 MAX485E, U3 STM32F103C8Tx, U4 AP1117-33, U5 ADuM1250AR, U6 L78L05_SOT89, U7 MCP4728, U8 LM358, U9 LM358, Y1 8MHz

Commit message: review AI V1 and AO V2
Parts:
- removed FB1: Ferrite_Bead, KiCAD_Additional_Parts:SMB-002, symbol Device:Ferrite_Bead
Connections:
- wire segments 563 -> 561
Changed lines of the file:
@@
 Text GLabel 2150 3850 0    50   Input ~ 0
 SCL
-Text GLabel 2150 3950 0    50   Input ~ 0
+Text GLabel 2150 3750 0    50   Input ~ 0
 SDA
 Wire Wire Line
-	2150 3950 2400 3950
+	2150 3750 2400 3750
 Wire Wire Line
 	2150 3850 2400 3850
@@
 NoConn ~ 2400 3550
 NoConn ~ 2400 3650
+NoConn ~ 2400 3950
 NoConn ~ 2400 4550
 NoConn ~ 2400 4650
@@
 F 3 "" H 4050 9650 50  0001 C CNN
 	1    4050 9650
+	1    0    0    -1
+$EndComp
+$Comp
+L Device:C C14
+U 1 1 62C1D340
+P 3550 9400
+F 0 "C14" H 3665 9446 50  0000 L CNN
+F 1 "1µ" H 3665 9355 50  0000 L CNN
+F 2 "Capacitor_SMD:C_0805_2012Metric_Pad1.18x1.45mm_HandSolder" H 3588 9250 50  0001 C CNN
+F 3 "~" H 3550 9400 50  0001 C CNN
+	1    3550 9400
 	1    0    0    -1
 $EndComp
@@
 	10750 10200 10750 10300
 Wire Wire Line
-	8150 8100 8300 8100
-Wire Wire Line
-	8150 8050 8150 8100
+	8500 8100 8700 8100
+Wire Wire Line
+	8500 8050 8500 8100
 $Comp
 L power:+24V #PWR042
 U 1 1 61553A60
-P 8150 8050
-F 0 "#PWR042" H 8150 7900 50  0001 C CNN
-F 1 "+24V" H 8165 8223 50  0000 C CNN
-F 2 "" H 8150 8050 50  0001 C CNN
-F 3 "" H 8150 8050 50  0001 C CNN
-	1    8150 8050
+P 8500 8050
+F 0 "#PWR042" H 8500 7900 50  0001 C CNN
+F 1 "+24V" H 8515 8223 50  0000 C CNN
+F 2 "" H 8500 8050 50  0001 C CNN
+F 3 "" H 8500 8050 50  0001 C CNN
+	1    8500 8050
 	1    0    0    -1
 $EndComp
@@
 Wire Wire Line
 	2200 8300 2650 8300
-NoConn ~ 2400 3750
-$Comp
-L Device:Ferrite_Bead FB1
-U 1 1 60E98E7C
-P 8500 8100
-F 0 "FB1" V 8226 8100 50  0000 C CNN
-F 1 "Ferrite_Bead" V 8317 8100 50  0000 C CNN
-F 2 "KiCAD_Additional_Parts:SMB-002" V 8430 8100 50  0001 C CNN
-F 3 "~" H 8500 8100 50  0001 C CNN
-	1    8500 8100
-	0    1    1    0
-$EndComp
-Wire Wire Line
-	8650 8100 8700 8100
-$Comp
-L power:PWR_FLAG #FLG02
-U 1 1 60EFDE96
-P 8300 8100
-F 0 "#FLG02" H 8300 8175 50  0001 C CNN
-F 1 "PWR_FLAG" H 8300 8273 50  0000 C CNN
-F 2 "" H 8300 8100 50  0001 C CNN
-F 3 "~" H 8300 8100 50  0001 C CNN
-	1    8300 8100
-	-1   0    0    1
-$EndComp
-Connection ~ 8300 8100
-Wire Wire Line
-	8300 8100 8350 8100
-$Comp
-L power:PWR_FLAG #FLG01
-U 1 1 60F006ED
-P 3150 9150
-F 0 "#FLG01" H 3150 9225 50  0001 C CNN
-F 1 "PWR_FLAG" H 3150 9323 50  0000 C CNN
-F 2 "" H 3150 9150 50  0001 C CNN
-F 3 "~" H 3150 9150 50  0001 C CNN
-	1    3150 9150
-	1    0    0    -1
-$EndComp
-Connection ~ 3150 9150
-$Comp
-L Device:C C14
-U 1 1 62C1D340
-P 3550 9400
-F 0 "C14" H 3665 9446 50  0000 L CNN
-F 1 "1µ" H 3665 9355 50  0000 L CNN
-F 2 "Capacitor_SMD:C_0805_2012Metric_Pad1.18x1.45mm_HandSolder" H 3588 9250 50  0001 C CNN
-F 3 "~" H 3550 9400 50  0001 C CNN
-	1    3550 9400
-	1    0    0    -1
-$EndComp
-$Comp
-L power:PWR_FLAG #FLG0101
-U 1 1 60F06704
-P 3550 9600
-F 0 "#FLG0101" H 3550 9675 50  0001 C CNN
-F 1 "PWR_FLAG" H 3550 9773 50  0000 C CNN
-F 2 "" H 3550 9600 50  0001 C CNN
-F 3 "~" H 3550 9600 50  0001 C CNN
-	1    3550 9600
-	-1   0    0    1
-$EndComp
-$Comp
-L power:PWR_FLAG #FLG0102
-U 1 1 60FD0830
-P 10750 10200
-F 0 "#FLG0102" H 10750 10275 50  0001 C CNN
-F 1 "PWR_FLAG" V 10750 10328 50  0000 L CNN
-F 2 "" H 10750 10200 50  0001 C CNN
-F 3 "~" H 10750 10200 50  0001 C CNN
-	1    10750 10200
-	0    1    1    0
-$EndComp
 $EndSCHEMATC
