File: pcbs/Platinen/kicad/AI_V1/AI_V1.kicad_pcb (KiCad board)
At the start: 4 copper layers, 100 x 77 mm, 126 parts, among them J1 Conn_01x04, J10 TBL009-500-02GY-2GY, J11 TBL009-500-02GY-2GY, J2 Conn_01x02, J3 Conn_01x02, J4 Conn_02x03_Odd_Even, J5 Conn_02x05_Odd_Even, J6 Conn_02x05_Odd_Even, J7 TBL009-500-02GY-2GY, J8 TBL009-500-02GY-2GY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

Commit message: update layout for AI
Parts:
- moved G*** 8.64 mm to (182.6, 76.2)
- moved C2 0.25 mm to (156.7, 128.5)
- moved C3 0.25 mm to (160.8, 128.5)
- moved R2 0.25 mm to (158.8, 126.5)
Routing:
- net GND2: vias 40 -> 63
- net GND: vias 15 -> 65
- added copper zone on In1.Cu, net GND
- added copper zone on In2.Cu, net GND
- added copper zone on B.Cu, net GND2
- added copper zone on In1.Cu, net GND2
- added copper zone on In2.Cu, net GND2
Other:
- board text added: "CAN"
- board text added: "RS485"

Commit message: review AI V1 and AO V2
Parts:
- added R44: 1k, Resistor_SMD:R_0805_2012Metric_Pad1.20x1.40mm_HandSolder, F.Cu at (123.5, 76.5)
- added R45: 1k, Resistor_SMD:R_0805_2012Metric_Pad1.20x1.40mm_HandSolder, F.Cu at (134.9, 76.5)
- added R46: 1k, Resistor_SMD:R_0805_2012Metric_Pad1.20x1.40mm_HandSolder, F.Cu at (146.3, 76.5)
- added R47: 1k, Resistor_SMD:R_0805_2012Metric_Pad1.20x1.40mm_HandSolder, F.Cu at (157.7, 76.5)
- added REF**: OSHW-Logo2_9.8x8mm_SilkScreen, Symbol:OSHW-Logo2_9.8x8mm_SilkScreen, F.Cu at (182.4, 92.2)
- C22, C23, C24, C25, C32, C33, C34, C35: value 10n -> 10p
- moved G*** 6.61 mm to (182.4, 69.6)
- moved R37 4.53 mm to (123.5, 74.4)
- moved R43 4.33 mm to (157.7, 74.4)
- moved R39 4.33 mm to (134.9, 74.4)
- moved R41 4.33 mm to (146.3, 74.4)
- moved R36 4.07 mm to (123.5, 72.4), turned to 180 degrees
- moved R38 4.06 mm to (134.9, 72.4), turned to 180 degrees
- moved R40 4.06 mm to (146.3, 72.4), turned to 180 degrees
- moved R42 4.06 mm to (157.7, 72.4), turned to 180 degrees
- moved FB2 2.17 mm to (138.7, 73.7), turned to 90 degrees
- moved FB3 2.17 mm to (150.1, 73.7), turned to 90 degrees
- moved FB4 2.17 mm to (161.5, 73.7), turned to 90 degrees
- moved FB1 1.93 mm to (127.3, 73.7), turned to 90 degrees
- moved C22 0.25 mm to (128.0, 89.7)
- moved J8 0.25 mm to (135.9, 67.8)
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Connections:
- FB1 pad 2: Net-(C38-Pad2) -> Net-(FB1-Pad2)
- FB2 pad 2: Net-(C39-Pad2) -> Net-(FB2-Pad2)
- FB3 pad 2: Net-(C40-Pad2) -> Net-(FB3-Pad2)
- FB4 pad 2: Net-(C41-Pad2) -> Net-(FB4-Pad2)
- R36 pad 1: Net-(C38-Pad2) -> Net-(FB1-Pad2)
- R38 pad 1: Net-(C39-Pad2) -> Net-(FB2-Pad2)
- R40 pad 1: Net-(C40-Pad2) -> Net-(FB3-Pad2)
- R42 pad 1: Net-(C41-Pad2) -> Net-(FB4-Pad2)
- U3 pad 41: SDA -> Net-(U3-Pad41)
- U3 pad 43: Net-(U3-Pad43) -> SDA
Routing:
- net Net-(FB2-Pad2): track 0.00 -> 10.7 mm
- net Net-(FB3-Pad2): track 0.00 -> 10.7 mm
- net Net-(FB1-Pad2): track 0.00 -> 10.7 mm
- net Net-(FB4-Pad2): track 0.00 -> 10.7 mm
- net Net-(Q2-Pad3): track 1.56 -> 7.43 mm
- net Net-(Q1-Pad3): track 1.56 -> 7.42 mm
- net Net-(Q4-Pad3): track 1.56 -> 7.32 mm
- net Net-(Q3-Pad3): track 1.56 -> 7.32 mm
- net Net-(C38-Pad2): track 10.5 -> 5.87 mm
- net Net-(C40-Pad2): track 10.5 -> 5.88 mm
- net Net-(C39-Pad2): track 10.5 -> 5.88 mm
- net Net-(C41-Pad2): track 10.5 -> 5.88 mm
- net Net-(D2-Pad3): track 12.6 -> 16.2 mm
- net Net-(D3-Pad3): track 12.6 -> 16.1 mm
- net Net-(D5-Pad3): track 12.6 -> 16.1 mm
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Other:
- board text added: "Marco Müller revved by theBrutzler"
- board text added: "SynPLC AI V1.0 16.06.21"
- board text removed: "SynPLC AI V1.0 14.06.21"

Commit message: bugfixes on PCBs
Parts:
- added C42: 1µ, Capacitor_SMD:C_0805_2012Metric_Pad1.18x1.45mm_HandSolder, F.Cu at (113.3, 86.6)
- added C43: 100n, Capacitor_SMD:C_0805_2012Metric_Pad1.18x1.45mm_HandSolder, F.Cu at (113.3, 84.6)
- added C44: 100n, Capacitor_SMD:C_0805_2012Metric_Pad1.18x1.45mm_HandSolder, F.Cu at (113.3, 75.4)
- added C45: 1µ, Capacitor_SMD:C_0805_2012Metric_Pad1.18x1.45mm_HandSolder, F.Cu at (113.3, 77.5)
- added D7: 1N4001, Diode_SMD:D_MELF, F.Cu at (109.2, 81.0)
- added U13: L78L10_SOT89, Package_TO_SOT_SMD:SOT-89-3, F.Cu at (113.8, 81.0)
- R20, R22, R24, R26: value 39k 0.1% -> 16k 0.1%
- R21, R23, R25, R27: value 16k 0.1% -> 11k 0.1%
- SW1: footprint Package_DIP:DIP-10_W7.62mm_Socket -> Button_Switch_THT:SW_DIP_SPSTx05_Slide_6.7x14.26mm_W7.62mm_P2.54mm_LowProfile
- moved J8 0.25 mm to (136.1, 67.8)
Connections:
- D2 pad 2: +24V -> +10V
- D3 pad 2: +24V -> +10V
- D4 pad 2: +24V -> +10V
- D5 pad 2: +24V -> +10V
Routing:
- net +10V: track 0.00 -> 70.0 mm, vias 0 -> 5
- net +24V: track 163.7 -> 140.7 mm, vias 13 -> 9

Commit message: started revs
Parts:
- added REF**: ESD-Logo_6.6x6mm_SilkScreen, Symbol:ESD-Logo_6.6x6mm_SilkScreen, F.Cu at (182.4, 99.7)
