File: pcbs/Platinen/kicad/AI_V1/AI_V1.sch (KiCad schematic (older format))
At the start: 129 parts, among them J1 Conn_01x04, J10 TBL009-500-02GY-2GY, J11 TBL009-500-02GY-2GY, J2 Conn_01x02, J3 Conn_01x02, J4 Conn_02x03_Odd_Even, J5 Conn_02x05_Odd_Even, J6 Conn_02x05_Odd_Even, J7 TBL009-500-02GY-2GY, J8 TBL009-500-02GY-2GY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

Commit message: bugfixes on PCBs
Parts:
- added C42, C45: 1µ, Capacitor_SMD:C_0805_2012Metric_Pad1.18x1.45mm_HandSolder, symbol Device:C
- added C43, C44: 100n, Capacitor_SMD:C_0805_2012Metric_Pad1.18x1.45mm_HandSolder, symbol Device:C
- added D7: 1N4001, Diode_SMD:D_MELF, symbol Diode:1N4001
- added U13: L78L10_SOT89, Package_TO_SOT_SMD:SOT-89-3, symbol Regulator_Linear:L78L05_SOT89
- R20, R22, R24, R26: value 39k 0.1% -> 16k 0.1%
- R21, R23, R25, R27: value 16k 0.1% -> 11k 0.1%
Connections:
- net +24V: now also C42.2, C43.2, D7.1 (K), U13.3 (IN); no longer D2.2, D3.2, D4.2, D5.2
- net GND2: now also C42.1, C43.1, C44.1, C45.1, U13.2 (GND)
- new net +10V: C44.2, C45.2, D2.2, D3.2, D4.2, D5.2, D7.2 (A), U13.1 (OUT)
- no-connect marks 16 -> 17
