File: pcbs/Platinen/kicad/AO_V2/AO_V2.kicad_pcb (KiCad board)
At the start: 4 copper layers, 100 x 77 mm, 157 parts, among them J1 Conn_01x04, J10 Conn_01x02, J11 Conn_01x02, J2 Conn_02x03_Odd_Even, J3 Conn_02x05_Odd_Even, J4 Conn_02x05_Odd_Even, J5 TBL009-500-02GY-2GY, J6 TBL009-500-02GY-2GY, J7 TBL009-500-02GY-2GY, J8 TBL009-500-02GY-2GY, J9 TBL009-500-02GY-2GY, K1 G6K-2, K2 G6K-2, K3 G6K-2, K4 G6K-2, Q1 BC846, Q2 BC846, Q3 BC846, Q4 BC846, SW1 SW_DIP_x05, U1 SN65HVD232, U10 LM358, U11 LM358, U2 MAX485E, U3 STM32F103C8Tx, U4 AP1117-33, U5 ADuM1250AR, U6 L78L05_SOT89, U7 MCP4728, U8 LM358, U9 LM358, Y1 8MHz

Commit message: review AI V1 and AO V2
Parts:
- added FB1: Ferrite_Bead, KiCAD_Additional_Parts:SMB-002, F.Cu at (99.6, 87.1)
- added REF**: OSHW-Logo2_9.8x8mm_SilkScreen, Symbol:OSHW-Logo2_9.8x8mm_SilkScreen, F.Cu at (175.0, 100.8)
- moved R3 4.84 mm to (143.7, 133.9)
- moved D5 3.10 mm to (96.5, 80.5)
- moved D6 3.10 mm to (101.1, 80.3)
- moved F1 3.10 mm to (101.3, 73.7)
Connections:
- D5 pad 1: +24V -> Net-(D5-Pad1)
- U3 pad 41: SDA -> Net-(U3-Pad41)
- U3 pad 43: Net-(U3-Pad43) -> SDA
Routing:
- net Net-(D5-Pad1): track 0.00 -> 7.79 mm
- net +24V: track 36.8 -> 43.6 mm, vias 12 -> 14
- net Net-(R3-Pad1): track 2.41 -> 7.25 mm
- net SDA: track 63.7 -> 66.9 mm
- net SCL: track 64.2 -> 66.3 mm
- net Net-(D6-Pad1): track 16.0 -> 17.7 mm
Other:
- board text added: "Marco Müller revved by theBrutzler"
- board text added: "SynPLC AO V2.0 16.06.21"
- board text removed: "SynPLC AO V2.0 13.06.21"

Commit message: started revs
Parts:
- added REF**: ESD-Logo_6.6x6mm_SilkScreen, Symbol:ESD-Logo_6.6x6mm_SilkScreen, F.Cu at (174.9, 108.5)
