File: pcbs/Platinen/kicad/DI8_V1.1/DI8_V1.1.kicad_pcb (KiCad board)
At the start: 4 copper layers, 100 x 77 mm, 157 parts, among them J1 Conn_01x04, J10 TBL009-500-02GY-2GY, J11 TBL009-500-02GY-2GY, J2 Conn_01x02, J3 Conn_01x02, J4 Conn_02x03_Odd_Even, J5 Conn_02x05_Odd_Even, J6 Conn_02x05_Odd_Even, J7 TBL009-500-02GY-2GY, J8 TBL009-500-02GY-2GY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

Commit message: finished layouts
Parts:
- moved REF** 5.59 mm to (129.5, 88.9)
Other:
- board text added: "485"
- board text added: "CAN"
- board text added: "Marco Müller not revved by theBrutzler yet"

Commit message: started revs
Routing:
- net CH1: track 127.8 -> 122.3 mm
- net CH2: track 115.3 -> 112.3 mm
- net CH5: track 47.1 -> 45.9 mm
- net CH4: track 86.6 -> 85.5 mm
- net GND2: vias 0 -> 31
- net GND: vias 55 -> 51

Commit message: complete reviews from dave
Parts:
- added REF**: ESD-Logo_6.6x6mm_SilkScreen, Symbol:ESD-Logo_6.6x6mm_SilkScreen, F.Cu at (129.5, 96.6)
Routing:
- net GND2: vias 31 -> 35
- net GND1: vias 0 -> 39
- net GND: vias 51 -> 52
Other:
- board text added: "Marco Müller revved by Blind_Via"
- board text removed: "Marco Müller not revved by theBrutzler yet"
