File: pcbs/Platinen/kicad/DI8_V1.1/DI8_V1.1.sch (KiCad schematic (older format))
At the start: 132 parts

Commit message: PCB update
Parts:
- added C1, C2: 20p, Capacitor_SMD:C_0805_2012Metric_Pad1.18x1.45mm_HandSolder, symbol Device:C
- added C10, C11, C12, C14, C3, C4, C6, C7, C8, C9: 100n, Capacitor_SMD:C_0805_2012Metric_Pad1.18x1.45mm_HandSolder, symbol Device:C
- added C13, C5: 1µ, Capacitor_SMD:C_0805_2012Metric_Pad1.18x1.45mm_HandSolder, symbol Device:C
- added J1: Conn_01x04, Connector_PinHeader_2.54mm:PinHeader_1x04_P2.54mm_Vertical, symbol Connector_Generic:Conn_01x04
- added J2, J3: Conn_01x02, Connector_PinHeader_2.54mm:PinHeader_1x02_P2.54mm_Vertical, symbol Connector_Generic:Conn_01x02
- added J4: Conn_02x03_Odd_Even, Connector_PinHeader_2.54mm:PinHeader_2x03_P2.54mm_Vertical, symbol Connector_Generic:Conn_02x03_Odd_Even
- added J5, J6: Conn_02x05_Odd_Even, Connector_PinHeader_2.54mm:PinHeader_2x05_P2.54mm_Horizontal, symbol Connector_Generic:Conn_02x05_Odd_Even
- added R1, R2: 1k, Resistor_SMD:R_0805_2012Metric_Pad1.20x1.40mm_HandSolder, symbol Device:R
- added R3: 1M, Resistor_SMD:R_0805_2012Metric_Pad1.20x1.40mm_HandSolder, symbol Device:R
- added R7: 120, Resistor_SMD:R_0805_2012Metric_Pad1.20x1.40mm_HandSolder, symbol Device:R
- added R8: 150, Resistor_SMD:R_0805_2012Metric_Pad1.20x1.40mm_HandSolder, symbol Device:R
- added U1: SN65HVD232, Package_SO:SOIC-8_3.9x4.9mm_P1.27mm, symbol Interface_CAN_LIN:SN65HVD232
- added U2: MAX485E, Package_SO:SOIC-8_3.9x4.9mm_P1.27mm, symbol Interface_UART:MAX485E
- added U4: AP1117-33, Package_TO_SOT_SMD:SOT-223-3_TabPin2, symbol Regulator_Linear:AP1117-33
- added Y1: 8MHz, Crystal:Crystal_SMD_HC49-SD, symbol Device:Crystal
- C15, C16, C17, C18, C19, C20, C21, C22, C23, C24, C25, C26, C27, C28, C29, C30: renamed from C?; footprint (none) -> Capacitor_SMD:C_0805_2012Metric_Pad1.18x1.45mm_HandSolder
- D1, D2, D3, D4, D5, D6, D7, D8: renamed from D?; footprint (none) -> LED_THT:LED_D3.0mm
- D10, D11, D12, D13, D14, D15, D16, D17, D18, D19, D20, D21, D22, D23, D24, D9: renamed from D?; footprint (none) -> Diode_SMD:D_MiniMELF
- FB1, FB2, FB3, FB4, FB5, FB6, FB7, FB8: renamed from FB?; footprint (none) -> KiCAD_Additional_Parts:SMB-001
- J10, J11, J7, J8, J9: renamed from J?; footprint TBL00950002GY2GY -> KiCAD_Additional_Parts:TBL00950002GY2GY; symbol KiCAD_personalized:TBL009-500-02GY-2GY -> DI8_V1.1-rescue:TBL009-500-02GY-2GY-KiCAD_personalized
- R10, R11, R12, R13, R14, R15, R16, R17, R18, R19, R20, R21, R22, R23, R24, R25, R26, R27, R28, R29, R30, R31, R32, R33, R34, R35, R36, R37, R38, R39, R4, R40, R41, R42, R43, R44, R45, R46, R47, R48, R49, R5, R50, R6, R9: renamed from R?; footprint (none) -> Resistor_SMD:R_0805_2012Metric_Pad1.20x1.40mm_HandSolder
- SW1: renamed from SW?; footprint (none) -> Button_Switch_THT:SW_DIP_SPSTx05_Slide_6.7x14.26mm_W7.62mm_P2.54mm_LowProfile
- gave numbers to parts that had none: 27
Connections:
- net labels added: BUS+, BUS-, CAN_RD, CAN_TD, DIR, RXD, TXD, VCC
- wire segments 302 -> 472
- no-connect marks 3 -> 15
Other:
- moved on the sheet: U5A, U5B, U5C, U5D, U6A, U6B, U6C, U6D

Commit message: started revs
Other:
- note added: "Galvanic Isolation\nmin. 1.5mm"
- note removed: "Galvanische Trennung\nmindestens 1,5mm"
Changed lines of the file:
@@
 Wire Notes Line
 	11200 3950 16050 3950
-Text Notes 11350 9050 1    50   ~ 0
-Galvanische Trennung\nmindestens 1,5mm
 $Comp
 L MCU_ST_STM32F1:STM32F103C8Tx U3
@@
 Wire Wire Line
 	7900 9150 8300 9150
-Text Notes 12750 3950 0    50   ~ 0
-Galvanische Trennung\nmindestens 1,5mm
+Text Notes 11400 9350 1    50   ~ 0
+Galvanic Isolation\nmin. 1.5mm
 $EndSCHEMATC
