File: pcbs/Platinen/kicad/DO8_V1.2/DO8_V1.2.sch (KiCad schematic (older format))
At the start: 82 parts

Commit message: PCB update
Parts:
- removed Q? (x7): BC846, Package_TO_SOT_SMD:SOT-23, symbol Transistor_BJT:BC846
- removed R? (x7): 2k2, symbol Device:R
- removed R? (x7): 1k, symbol Device:R
- added C1, C10, C11, C12, C13, C14, C15, C3, C4, C6, C7, C8, C9: 100n, Capacitor_SMD:C_0805_2012Metric_Pad1.18x1.45mm_HandSolder, symbol Device:C
- added C2, C5: 1µ, Capacitor_SMD:C_0805_2012Metric_Pad1.18x1.45mm_HandSolder, symbol Device:C
- added D1, D10, D12, D15, D2, D3, D4, D7: LED, LED_THT:LED_D3.0mm, symbol Device:LED
- added J1: Conn_01x04, Connector_PinHeader_2.54mm:PinHeader_1x04_P2.54mm_Vertical, symbol Connector_Generic:Conn_01x04
- added J2, J3: Conn_01x02, Connector_PinHeader_2.54mm:PinHeader_1x02_P2.54mm_Vertical, symbol Connector_Generic:Conn_01x02
- added J4: Conn_02x03_Odd_Even, Connector_PinHeader_2.54mm:PinHeader_2x03_P2.54mm_Vertical, symbol Connector_Generic:Conn_02x03_Odd_Even
- added J5, J6: Conn_02x05_Odd_Even, Connector_PinHeader_2.54mm:PinHeader_2x05_P2.54mm_Horizontal, symbol Connector_Generic:Conn_02x05_Odd_Even
- added Q2, Q3, Q4, Q5, Q6, Q7, Q8: BC846, Package_TO_SOT_SMD:SOT-23, symbol Transistor_BJT:BC846
- added R10, R11, R12, R13, R14, R15, R16, R32, R35, R37, R39, R41, R43, R45, R47, R50, R51: 1k, Resistor_SMD:R_0805_2012Metric_Pad1.20x1.40mm_HandSolder, symbol Device:R
- added R18, R19, R20, R21, R22, R23, R24: 2k2, Resistor_SMD:R_0805_2012Metric_Pad1.20x1.40mm_HandSolder, symbol Device:R
- added R2: 120, Resistor_SMD:R_0805_2012Metric_Pad1.20x1.40mm_HandSolder, symbol Device:R
- added R3: 150, Resistor_SMD:R_0805_2012Metric_Pad1.20x1.40mm_HandSolder, symbol Device:R
- added U1: SN65HVD232, Package_SO:SOIC-8_3.9x4.9mm_P1.27mm, symbol Interface_CAN_LIN:SN65HVD232
- added U2: MAX485E, Package_SO:SO-8_3.9x4.9mm_P1.27mm, symbol Interface_UART:MAX485E
- added U4: AP1117-33, Package_TO_SOT_SMD:SOT-223-3_TabPin2, symbol Regulator_Linear:AP1117-33
- added Y1: 8MHz, Crystal:Crystal_SMD_HC49-SD, symbol Device:Crystal
- D17: renamed from D?; footprint (none) -> Diode_SMD:D_MiniMELF
- IC1: renamed from IC?; footprint PG-DSO-36 -> KiCAD_Additional_Parts:PG-DSO-36
- J10, J11, J7, J8, J9: renamed from J?; footprint TBL00950002GY2GY -> KiCAD_Additional_Parts:TBL00950002GY2GY; symbol KiCAD_personalized:TBL009-500-02GY-2GY -> DO8_V1.2-rescue:TBL009-500-02GY-2GY-KiCAD_personalized
- R1, R17, R25, R26, R27, R28, R29, R30, R31, R33, R34, R36, R38, R4, R40, R42, R44, R46, R48, R49, R5, R6, R7, R8, R9: renamed from R?; footprint (none) -> Resistor_SMD:R_0805_2012Metric_Pad1.20x1.40mm_HandSolder
- SW1: renamed from SW?; footprint (none) -> Button_Switch_THT:SW_DIP_SPSTx05_Slide_9.78x14.88mm_W7.62mm_P2.54mm
- gave numbers to parts that had none: 16
Connections:
- net labels added: BUS+, BUS-, CAN_RD, CAN_TD, DIR, RXD, TXD
- wire segments 273 -> 449
- no-connect marks 4 -> 8
Other:
- note added: "Galvanische Trennung\nmindestens 1,5mm\n"
- moved on the sheet: U7A, U7B, U7C, U7D, U8A, U8B, U8C, U8D

Commit message: finished layouts
Parts:
- added D19, D20, D21, D22, D23, D24, D25, D26: LL4148, Diode_SMD:D_MiniMELF, symbol Diode:LL4148
Connections:
- net at D16.1 (A1), IC1.21 (OUT8@2), IC1.22 (OUT8)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: now also D26.2 (A); no longer R48.1
- net at D14.1 (A1), IC1.23 (OUT7@2), IC1.24 (OUT7)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: now also D25.2 (A); no longer R46.1
- net at D13.1 (A1), IC1.25 (OUT6@2), IC1.26 (OUT6)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: now also D24.2 (A); no longer R44.1
- net at D11.1 (A1), IC1.27 (OUT5@2), IC1.28 (OUT5)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: now also D23.2 (A); no longer R42.1
- net at D9.1 (A1), IC1.29 (OUT4@2), IC1.30 (OUT4)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: now also D22.2 (A); no longer R40.1
- net at D8.1 (A1), IC1.31 (OUT3@2), IC1.32 (OUT3)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: now also D21.2 (A); no longer R38.1
- net at D6.1 (A1), IC1.33 (OUT2@2), IC1.34 (OUT2)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: now also D20.2 (A); no longer R36.1
- net at D5.1 (A1), IC1.35 (OUT1@2), IC1.36 (OUT1)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: now also D19.2 (A); no longer R34.1
- new net: D19.1 (K), R34.1
- new net: D20.1 (K), R36.1
- new net: D21.1 (K), R38.1
- new net: D22.1 (K), R40.1
- new net: D23.1 (K), R42.1
- new net: D24.1 (K), R44.1
- new net: D25.1 (K), R46.1
- new net: D26.1 (K), R48.1
Changed lines of the file:
@@
 	13850 4900 14100 4900
 Wire Wire Line
-	14100 4900 14100 5750
+	14100 4900 14100 5200
 Connection ~ 14000 3100
 Wire Wire Line
@@
 	13700 3100 13700 3150
 Wire Wire Line
-	13550 3100 13550 5750
+	13550 3100 13550 5200
 Wire Wire Line
 	13400 3100 13250 3100
@@
 	13250 4900 13000 4900
 Wire Wire Line
-	13000 4900 13000 5750
+	13000 4900 13000 5200
 Connection ~ 13400 3100
 Wire Wire Line
 	13400 3100 13400 3150
 Wire Wire Line
-	12450 5750 12450 4900
+	12450 5750 12450 5500
 Wire Wire Line
 	12450 4900 12950 4900
@@
 	12650 4850 11900 4850
 Wire Wire Line
-	11900 4850 11900 5750
+	11900 4850 11900 5200
 Connection ~ 12800 3100
 Wire Wire Line
@@
 	12350 4800 11350 4800
 Wire Wire Line
-	11350 4800 11350 5750
+	11350 4800 11350 5200
 Connection ~ 12500 3100
 Wire Wire Line
@@
 	12050 4750 10800 4750
 Wire Wire Line
-	10800 4750 10800 5750
+	10800 4750 10800 5200
 Connection ~ 12200 3100
 Wire Wire Line
@@
 	11750 4700 10250 4700
 Wire Wire Line
-	10250 4700 10250 5750
+	10250 4700 10250 5200
 Connection ~ 11900 3100
 Wire Wire Line
@@
 	1    0    0    -1
 $EndComp
+$Comp
+L Diode:LL4148 D19
+U 1 1 60EA1319
+P 10250 5350
+F 0 "D19" V 10296 5270 50  0000 R CNN
+F 1 "LL4148" V 10205 5270 50  0000 R CNN
+F 2 "Diode_SMD:D_MiniMELF" H 10250 5175 50  0001 C CNN
+F 3 "http://www.vishay.com/docs/85557/ll4148.pdf" H 10250 5350 50  0001 C CNN
+	1    10250 5350
+	0    -1   -1   0
+$EndComp
+Wire Wire Line
+	10250 5500 10250 5750
+$Comp
+L Diode:LL4148 D20
+U 1 1 60EA3837
+P 10800 5350
+F 0 "D20" V 10846 5270 50  0000 R CNN
+F 1 "LL4148" V 10755 5270 50  0000 R CNN
+F 2 "Diode_SMD:D_MiniMELF" H 10800 5175 50  0001 C CNN
+F 3 "http://www.vishay.com/docs/85557/ll4148.pdf" H 10800 5350 50  0001 C CNN
+	1    10800 5350
+	0    -1   -1   0
+$EndComp
+Wire Wire Line
+	10800 5500 10800 5750
+$Comp
+L Diode:LL4148 D21
+U 1 1 60EA3CF3
+P 11350 5350
+F 0 "D21" V 11396 5270 50  0000 R CNN
+F 1 "LL4148" V 11305 5270 50  0000 R CNN
+F 2 "Diode_SMD:D_MiniMELF" H 11350 5175 50  0001 C CNN
+F 3 "http://www.vishay.com/docs/85557/ll4148.pdf" H 11350 5350 50  0001 C CNN
+	1    11350 5350
+	0    -1   -1   0
+$EndComp
+Wire Wire Line
+	11350 5500 11350 5750
+$Comp
+L Diode:LL4148 D22
+U 1 1 60EA42EA
+P 11900 5350
+F 0 "D22" V 11946 5270 50  0000 R CNN
+F 1 "LL4148" V 11855 5270 50  0000 R CNN
+F 2 "Diode_SMD:D_MiniMELF" H 11900 5175 50  0001 C CNN
+F 3 "http://www.vishay.com/docs/85557/ll4148.pdf" H 11900 5350 50  0001 C CNN
+	1    11900 5350
+	0    -1   -1   0
+$EndComp
+Wire Wire Line
+	11900 5500 11900 5750
+$Comp
+L Diode:LL4148 D23
+U 1 1 60EA49D4
+P 12450 5350
+F 0 "D23" V 12496 5270 50  0000 R CNN
+F 1 "LL4148" V 12405 5270 50  0000 R CNN
+F 2 "Diode_SMD:D_MiniMELF" H 12450 5175 50  0001 C CNN
+F 3 "http://www.vishay.com/docs/85557/ll4148.pdf" H 12450 5350 50  0001 C CNN
+	1    12450 5350
+	0    -1   -1   0
+$EndComp
+Wire Wire Line
+	12450 5200 12450 4900
+$Comp
+L Diode:LL4148 D24
+U 1 1 60EA4F2A
+P 13000 5350
+F 0 "D24" V 13046 5270 50  0000 R CNN
+F 1 "LL4148" V 12955 5270 50  0000 R CNN
+F 2 "Diode_SMD:D_MiniMELF" H 13000 5175 50  0001 C CNN
+F 3 "http://www.vishay.com/docs/85557/ll4148.pdf" H 13000 5350 50  0001 C CNN
+	1    13000 5350
+	0    -1   -1   0
+$EndComp
+Wire Wire Line
+	13000 5500 13000 5750
+$Comp
+L Diode:LL4148 D25
+U 1 1 60EA55F9
+P 13550 5350
+F 0 "D25" V 13596 5270 50  0000 R CNN
+F 1 "LL4148" V 13505 5270 50  0000 R CNN
+F 2 "Diode_SMD:D_MiniMELF" H 13550 5175 50  0001 C CNN
+F 3 "http://www.vishay.com/docs/85557/ll4148.pdf" H 13550 5350 50  0001 C CNN
+	1    13550 5350
+	0    -1   -1   0
+$EndComp
+Wire Wire Line
+	13550 5500 13550 5750
+$Comp
+L Diode:LL4148 D26
+U 1 1 60EA5BFC
+P 14100 5350
+F 0 "D26" V 14146 5270 50  0000 R CNN
+F 1 "LL4148" V 14055 5270 50  0000 R CNN
+F 2 "Diode_SMD:D_MiniMELF" H 14100 5175 50  0001 C CNN
+F 3 "http://www.vishay.com/docs/85557/ll4148.pdf" H 14100 5350 50  0001 C CNN
+	1    14100 5350
+	0    -1   -1   0
+$EndComp
+Wire Wire Line
+	14100 5500 14100 5750
 $EndSCHEMATC
