File: pcbs/Platinen/kicad/XP_V1/XP_V1.sch (KiCad schematic (older format))
At the start: 8 parts

Commit message: greate gerbers, plot schematics
Other:
- moved on the sheet: Q?, R?
Changed lines of the file:
@@
 EELAYER 30 0
 EELAYER END
-$Descr A3 16535 11693
+$Descr A3 11693 16535 portrait
 encoding utf-8
 Sheet 1 1
@@
 L Transistor_BJT:BC856 Q?
 U 1 1 60ED5FBE
-P 11400 1100
-F 0 "Q?" H 11591 1054 50  0000 L CNN
-F 1 "BC856" H 11591 1145 50  0000 L CNN
-F 2 "Package_TO_SOT_SMD:SOT-23" H 11600 1025 50  0001 L CIN
-F 3 "https://www.onsemi.com/pub/Collateral/BC860-D.pdf" H 11400 1100 50  0001 L CNN
-	1    11400 1100
+P 9600 1100
+F 0 "Q?" H 9791 1054 50  0000 L CNN
+F 1 "BC856" H 9791 1145 50  0000 L CNN
+F 2 "Package_TO_SOT_SMD:SOT-23" H 9800 1025 50  0001 L CIN
+F 3 "https://www.onsemi.com/pub/Collateral/BC860-D.pdf" H 9600 1100 50  0001 L CNN
+	1    9600 1100
 	1    0    0    1
 $EndComp
@@
 L Transistor_BJT:BC846 Q?
 U 1 1 60ED6B2C
-P 11050 1700
-F 0 "Q?" H 11241 1746 50  0000 L CNN
-F 1 "BC846" H 11241 1655 50  0000 L CNN
-F 2 "Package_TO_SOT_SMD:SOT-23" H 11250 1625 50  0001 L CIN
-F 3 "https://assets.nexperia.com/documents/data-sheet/BC846_SER.pdf" H 11050 1700 50  0001 L CNN
-	1    11050 1700
+P 9250 1700
+F 0 "Q?" H 9441 1746 50  0000 L CNN
+F 1 "BC846" H 9441 1655 50  0000 L CNN
+F 2 "Package_TO_SOT_SMD:SOT-23" H 9450 1625 50  0001 L CIN
+F 3 "https://assets.nexperia.com/documents/data-sheet/BC846_SER.pdf" H 9250 1700 50  0001 L CNN
+	1    9250 1700
 	1    0    0    -1
 $EndComp
@@
 L Device:Q_NMOS_GDS Q?
 U 1 1 60ED8AED
-P 11850 1350
-F 0 "Q?" H 12054 1396 50  0000 L CNN
-F 1 "BUK98150-55A/CUF " H 12054 1305 50  0000 L CNN
-F 2 "" H 12050 1450 50  0001 C CNN
-F 3 "~" H 11850 1350 50  0001 C CNN
-	1    11850 1350
+P 10050 1350
+F 0 "Q?" H 10254 1396 50  0000 L CNN
+F 1 "BUK98150-55A/CUF " H 10254 1305 50  0000 L CNN
+F 2 "" H 10250 1450 50  0001 C CNN
+F 3 "~" H 10050 1350 50  0001 C CNN
+	1    10050 1350
 	1    0    0    -1
 $EndComp
@@
 L Device:R R?
 U 1 1 60ED9F27
-P 11150 1300
-F 0 "R?" H 11220 1346 50  0000 L CNN
-F 1 "1k" H 11220 1255 50  0000 L CNN
-F 2 "" V 11080 1300 50  0001 C CNN
-F 3 "~" H 11150 1300 50  0001 C CNN
-	1    11150 1300
+P 9350 1300
+F 0 "R?" H 9420 1346 50  0000 L CNN
+F 1 "1k" H 9420 1255 50  0000 L CNN
+F 2 "" V 9280 1300 50  0001 C CNN
+F 3 "~" H 9350 1300 50  0001 C CNN
+	1    9350 1300
 	1    0    0    -1
 $EndComp
@@
 L Device:R R?
 U 1 1 60EDA1E9
-P 11150 900
-F 0 "R?" H 11220 946 50  0000 L CNN
-F 1 "1k" H 11220 855 50  0000 L CNN
-F 2 "" V 11080 900 50  0001 C CNN
-F 3 "~" H 11150 900 50  0001 C CNN
-	1    11150 900
-	1    0    0    -1
-$EndComp
-Wire Wire Line
-	11500 900  11500 700
+P 9350 900
+F 0 "R?" H 9420 946 50  0000 L CNN
+F 1 "1k" H 9420 855 50  0000 L CNN
+F 2 "" V 9280 900 50  0001 C CNN
+F 3 "~" H 9350 900 50  0001 C CNN
+	1    9350 900
+	1    0    0    -1
+$EndComp
+Wire Wire Line
+	9700 900  9700 700
 $Comp
 L power:GND1 #PWR?
 U 1 1 60EE09E8
-P 11950 1550
-F 0 "#PWR?" H 11950 1300 50  0001 C CNN
-F 1 "GND1" H 11955 1377 50  0000 C CNN
-F 2 "" H 11950 1550 50  0001 C CNN
-F 3 "" H 11950 1550 50  0001 C CNN
-	1    11950 1550
+P 10150 1550
+F 0 "#PWR?" H 10150 1300 50  0001 C CNN
+F 1 "GND1" H 10155 1377 50  0000 C CNN
+F 2 "" H 10150 1550 50  0001 C CNN
+F 3 "" H 10150 1550 50  0001 C CNN
+	1    10150 1550
 	1    0    0    -1
 $EndComp
@@
 L power:GND1 #PWR?
 U 1 1 60EE0E4F
-P 11150 1900
-F 0 "#PWR?" H 11150 1650 50  0001 C CNN
-F 1 "GND1" H 11155 1727 50  0000 C CNN
-F 2 "" H 11150 1900 50  0001 C CNN
-F 3 "" H 11150 1900 50  0001 C CNN
-	1    11150 1900
-	1    0    0    -1
-$EndComp
-Wire Wire Line
-	11950 700  11950 1150
-Wire Wire Line
-	11150 700  11150 750
-Wire Wire Line
-	11150 700  11500 700
-Wire Wire Line
-	11150 1500 11150 1450
-Wire Wire Line
-	11150 1150 11150 1100
-Wire Wire Line
-	11150 1100 11200 1100
-Connection ~ 11150 1100
-Wire Wire Line
-	11150 1100 11150 1050
-Text GLabel 12150 700  2    50   Input ~ 0
+P 9350 1900
+F 0 "#PWR?" H 9350 1650 50  0001 C CNN
+F 1 "GND1" H 9355 1727 50  0000 C CNN
+F 2 "" H 9350 1900 50  0001 C CNN
+F 3 "" H 9350 1900 50  0001 C CNN
+	1    9350 1900
+	1    0    0    -1
+$EndComp
+Wire Wire Line
+	10150 700  10150 1150
+Wire Wire Line
+	9350 700  9350 750
+Wire Wire Line
+	9350 700  9700 700
+Wire Wire Line
+	9350 1500 9350 1450
+Wire Wire Line
+	9350 1150 9350 1100
+Wire Wire Line
+	9350 1100 9400 1100
+Connection ~ 9350 1100
+Wire Wire Line
+	9350 1100 9350 1050
+Text GLabel 10350 700  2    50   Input ~ 0
 OD1
 Wire Wire Line
-	12150 700  11950 700
-Text GLabel 10450 1700 0    50   Input ~ 0
+	10350 700  10150 700
+Text GLabel 8650 1700 0    50   Input ~ 0
 PWM1
 Wire Wire Line
-	10800 1700 10850 1700
+	9000 1700 9050 1700
 $Comp
 L Device:R R?
 U 1 1 60EEB567
-P 11500 1550
-F 0 "R?" H 11570 1596 50  0000 L CNN
-F 1 "1k" H 11570 1505 50  0000 L CNN
-F 2 "" V 11430 1550 50  0001 C CNN
-F 3 "~" H 11500 1550 50  0001 C CNN
-	1    11500 1550
+P 9700 1550
+F 0 "R?" H 9770 1596 50  0000 L CNN
+F 1 "1k" H 9770 1505 50  0000 L CNN
+F 2 "" V 9630 1550 50  0001 C CNN
+F 3 "~" H 9700 1550 50  0001 C CNN
+	1    9700 1550
 	1    0    0    -1
 $EndComp
@@
 L power:GND1 #PWR?
 U 1 1 60EEBEE9
-P 11500 1750
-F 0 "#PWR?" H 11500 1500 50  0001 C CNN
-F 1 "GND1" H 11505 1577 50  0000 C CNN
-F 2 "" H 11500 1750 50  0001 C CNN
-F 3 "" H 11500 1750 50  0001 C CNN
-	1    11500 1750
-	1    0    0    -1
-$EndComp
-Wire Wire Line
-	11500 1750 11500 1700
-Wire Wire Line
-	11500 1400 11500 1350
-Wire Wire Line
-	11650 1350 11500 1350
-Connection ~ 11500 1350
-Wire Wire Line
-	11500 1350 11500 1300
+P 9700 1750
+F 0 "#PWR?" H 9700 1500 50  0001 C CNN
+F 1 "GND1" H 9705 1577 50  0000 C CNN
+F 2 "" H 9700 1750 50  0001 C CNN
+F 3 "" H 9700 1750 50  0001 C CNN
+	1    9700 1750
+	1    0    0    -1
+$EndComp
+Wire Wire Line
+	9700 1750 9700 1700
+Wire Wire Line
+	9700 1400 9700 1350
+Wire Wire Line
+	9850 1350 9700 1350
+Connection ~ 9700 1350
+Wire Wire Line
+	9700 1350 9700 1300
 $Comp
 L Device:R R?
 U 1 1 60EF2CBC
-P 10650 1700
-F 0 "R?" V 10443 1700 50  0000 C CNN
-F 1 "1k" V 10534 1700 50  0000 C CNN
-F 2 "" V 10580 1700 50  0001 C CNN
-F 3 "~" H 10650 1700 50  0001 C CNN
-	1    10650 1700
+P 8850 1700
+F 0 "R?" V 8643 1700 50  0000 C CNN
+F 1 "1k" V 8734 1700 50  0000 C CNN
+F 2 "" V 8780 1700 50  0001 C CNN
+F 3 "~" H 8850 1700 50  0001 C CNN
+	1    8850 1700
 	0    1    1    0
 $EndComp
 Wire Wire Line
-	10450 1700 10500 1700
-Text GLabel 12150 2200 2    50   Input ~ 0
+	8650 1700 8700 1700
+Text GLabel 10350 2200 2    50   Input ~ 0
 OD3
-Text GLabel 10450 3200 0    50   Input ~ 0
+Text GLabel 8650 3200 0    50   Input ~ 0
 PWM3
 Wire Wire Line
-	10450 3200 10500 3200
-Text GLabel 12150 3700 2    50   Input ~ 0
+	8650 3200 8700 3200
+Text GLabel 10350 3700 2    50   Input ~ 0
 OD5
-Text GLabel 10450 4700 0    50   Input ~ 0
+Text GLabel 8650 4700 0    50   Input ~ 0
 PWM5
 Wire Wire Line
-	10450 4700 10500 4700
-Text GLabel 12150 5200 2    50   Input ~ 0
+	8650 4700 8700 4700
+Text GLabel 10350 5200 2    50   Input ~ 0
 OD7
-Text GLabel 10450 6200 0    50   Input ~ 0
+Text GLabel 8650 6200 0    50   Input ~ 0
 PWM7
 Wire Wire Line
-	10450 6200 10500 6200
-Text GLabel 15050 650  2    50   Input ~ 0
+	8650 6200 8700 6200
+Text GLabel 10400 8200 2    50   Input ~ 0
 OD2
-Text GLabel 13350 1650 0    50   Input ~ 0
+Text GLabel 8700 9200 0    50   Input ~ 0
 PWM2
 Wire Wire Line
-	13350 1650 13400 1650
-Text GLabel 15050 2150 2    50   Input ~ 0
+	8700 9200 8750 9200
+Text GLabel 10400 9700 2    50   Input ~ 0
 OD4
-Text GLabel 13350 3150 0    50   Input ~ 0
+Text GLabel 8700 10700 0    50   Input ~ 0
 PWM4
 Wire Wire Line
-	13350 3150 13400 3150
-Text GLabel 15050 3650 2    50   Input ~ 0
+	8700 10700 8750 10700
+Text GLabel 10400 11200 2    50   Input ~ 0
 OD6
-Text GLabel 13350 4650 0    50   Input ~ 0
+Text GLabel 8700 12200 0    50   Input ~ 0
 PWM6
 Wire Wire Line
-	13350 4650 13400 4650
-Text GLabel 15050 5150 2    50   Input ~ 0
+	8700 12200 8750 12200
+Text GLabel 10400 12700 2    50   Input ~ 0
 OD8
-Text GLabel 13350 6150 0    50   Input ~ 0
+Text GLabel 8700 13700 0    50   Input ~ 0
 PWM8
 Wire Wire Line
-	13350 6150 13400 6150
+	8700 13700 8750 13700
 $Comp
 L power:+5V #PWR?
 U 1 1 60F89F98
-P 11600 700
-F 0 "#PWR?" H 11600 550 50  0001 C CNN
-F 1 "+5V" V 11615 828 50  0000 L CNN
-F 2 "" H 11600 700 50  0001 C CNN
-F 3 "" H 11600 700 50  0001 C CNN
-	1    11600 700
+P 9800 700
+F 0 "#PWR?" H 9800 550 50  0001 C CNN
+F 1 "+5V" V 9815 828 50  0000 L CNN
+F 2 "" H 9800 700 50  0001 C CNN
+F 3 "" H 9800 700 50  0001 C CNN
+	1    9800 700
 	0    1    1    0
 $EndComp
 Wire Wire Line
-	11600 700  11500 700
-Connection ~ 11500 700
+	9800 700  9700 700
+Connection ~ 9700 700
 $EndSCHEMATC
