File: pcbs/Platinen/kicad/CPU_V2/CPU_V2/CPU_V2.kicad_pcb (KiCad board)
At the start: 4 copper layers, 100 x 77 mm, 115 parts, among them J2 SWD, J4 24V_In, J5 Conn_02x05_Odd_Even, J6 Conn_02x03_Odd_Even, J7 SPI Conn, Q1 BSS138, Q2 BSS138, Q3 BSS138, Q4 BC856, Q5 BSS138, Q6 BSS138, U1 STM32F412RETx, U2 THN 10-2411WIR, U3 AP1117-33, U4 MAX485E, U5 SN65HVD232, U6 ESP-01, Y1 12MHz, Y2 32.768kHz

Commit message: CPU Update Finish CPU V2 Design and finish CPU PiggyBack Board
Parts:
- added C35: 1µ, Capacitor_SMD:C_0805_2012Metric, F.Cu at (90.3, 114.3)
- added G***: LOGO, eigene:logo, F.Cu at (148.7, 126.6)
- added J1: GSD09002SEU, eigene:GSD09002SEU, F.Cu at (153.6, 96.4)
- added J3: USB_B, Connector_USB:USB_B_Lumberg_2411_02_Horizontal, F.Cu at (170.3, 128.8)
- added J8: I2C, Connector_PinHeader_2.54mm:PinHeader_1x04_P2.54mm_Vertical, F.Cu at (87.4, 114.4)
- added Q7: BSS138, Package_TO_SOT_SMD:SOT-23, F.Cu at (105.4, 109.9)
- added Q8: BSS138, Package_TO_SOT_SMD:SOT-23, F.Cu at (105.4, 106.4)
- added R12: 10k, Resistor_SMD:R_0805_2012Metric, F.Cu at (150.6, 102.4)
- added R13: 10k, Resistor_SMD:R_0805_2012Metric, F.Cu at (150.6, 118.1)
- added R47: 4k7, Resistor_SMD:R_0805_2012Metric, F.Cu at (108.5, 109.9)
- added R48: 4k7, Resistor_SMD:R_0805_2012Metric, F.Cu at (102.4, 109.9)
- added R49: 4k7, Resistor_SMD:R_0805_2012Metric, F.Cu at (108.5, 106.4)
- added R50: 4k7, Resistor_SMD:R_0805_2012Metric, F.Cu at (102.4, 106.4)
- added REF**: ESD-Logo_6.6x6mm_SilkScreen, Symbol:ESD-Logo_6.6x6mm_SilkScreen, F.Cu at (125.1, 127.5)
- added REF**: OSHW-Logo2_9.8x8mm_SilkScreen, Symbol:OSHW-Logo2_9.8x8mm_SilkScreen, F.Cu at (142.1, 134.6)
- moved C24 159.1 mm to (87.1, 101.1), turned to 180 degrees
- moved C23 148.4 mm to (87.1, 99.1), turned to 180 degrees
- moved C26 137.3 mm to (91.7, 99.1)
- moved C25 130.5 mm to (91.7, 101.1)
- moved R34 123.7 mm to (157.5, 135.6), turned to -90 degrees
- moved R6 120.1 mm to (147.1, 109.0)
- moved R36 114.2 mm to (162.3, 132.8), turned to 180 degrees
- moved R29 113.3 mm to (139.4, 84.8), turned to 90 degrees
- moved R17 112.5 mm to (149.6, 65.0), turned to 90 degrees
- moved R15 111.2 mm to (150.6, 98.0)
- moved R30 111.0 mm to (139.4, 90.9), turned to 90 degrees
- moved R9 110.0 mm to (139.4, 66.5), turned to 90 degrees
- moved R26 106.7 mm to (150.6, 114.8)
- moved D5 105.8 mm to (142.7, 86.1), turned to 90 degrees
- moved R14 104.2 mm to (150.6, 95.5)
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- renumbered R12 to R14, R13 to R15, R14 to R16, R15 to R17, R16 to R18, R17 to R19, R18 to R20, R20 to R21, R21 to R22, R22 to R23, R19 to R24, R24 to R25, R23 to R26, R25 to R27, R26 to R28, R27 to R29, R28 to R30, R29 to R31, R30 to R32, R31 to R33, R32 to R34, R33 to R35, R34 to R36, R35 to R37, R36 to R38, R37 to R39, R38 to R40, R39 to R41, R40 to R42, R41 to R43, R42 to R44, R43 to R45, R44 to R46
Connections:
- net Net-(J3-Pad2) renamed /D-
- net Net-(J3-Pad3) renamed /D+
- net USB_DM- renamed USB-
- net USB_DP+ renamed USB+
- J5 pad 1: VCC -> +5V
- J5 pad 2: VCC -> +5V
- J5 pad 3: VCC -> +5V
- J5 pad 4: VCC -> +5V
- U1 pad 20: unconnected-(U1-Pad20) -> SDIO_CardDetect
- U1 pad 21: unconnected-(U1-Pad21) -> SDIO_WriteProtect
- U1 pad 53: unconnected-(U1-Pad53) -> LED_BOOT
- U1 pad 54: unconnected-(U1-Pad54) -> LED_HEARTBEAT
- U1 pad 58: LED_HEARTBEAT -> I2C1_SCL
- U1 pad 59: LED_BOOT -> I2C1_SDA
Routing:
- net GND: track 0.00 -> 174.5 mm, vias 0 -> 129
- net +5V: track 0.00 -> 128.5 mm, vias 0 -> 12
- net +3V3: track 0.00 -> 97.3 mm, vias 0 -> 28
- net SPI2_SCK: track 0.00 -> 75.9 mm, vias 0 -> 1
- net SPI2_MOSI: track 0.00 -> 72.6 mm, vias 0 -> 2
- net SPI2_MISO: track 0.00 -> 69.8 mm, vias 0 -> 2
- net SPI_CS1: track 0.00 -> 64.6 mm, vias 0 -> 1
- net USART2_RX: track 0.00 -> 64.0 mm, vias 0 -> 2
- net LED_ERROR: track 0.00 -> 62.9 mm, vias 0 -> 2
- net LED_RUN: track 0.00 -> 57.0 mm, vias 0 -> 2
- net USART2_TX: track 0.00 -> 55.9 mm, vias 0 -> 3
- net LED_FLASH: track 0.00 -> 51.1 mm, vias 0 -> 2
- net LED_HEARTBEAT: track 0.00 -> 42.7 mm, vias 0 -> 2
- net USB+: track 0.00 -> 42.1 mm, vias 0 -> 2
- net /VBAT: track 0.00 -> 40.8 mm
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- added copper zone on In2.Cu, net +3V3
- added copper zone on F.Cu, net +5V
- added copper zone on In2.Cu, net +5V
- added copper zone on B.Cu, net GND
- added copper zone on F.Cu, net GND
- added copper zone on In1.Cu, net GND
Other:
- board text added: "+"
- board text added: "5V USB"
- board text added: "CAN"
- board text added: "GND 5V SDA SCL"
- board text added: "GND SWCLK SWDIO 3V3"
- board text added: "JLCJLCJLC"
- board text added: "RS485"
- board text added: "SynPLC CPU V2"
