File: pcbs/Platinen/kicad/CPU_V2/CPU_V2/CPU_V2.kicad_sch (KiCad schematic)
At the start: 117 parts, among them J1 Micro_SD_Card, J2 SWD, J3 USB_B_Micro, J4 24V_In, J5 Conn_02x05_Odd_Even, J6 Conn_02x03_Odd_Even, J7 SPI Conn, Q1 BSS138, Q2 BSS138, Q3 BSS138, Q4 BC856, Q5 BSS138, Q6 BSS138, U1 STM32F412RETx, U2 THN 10-2411WIR, U3 AP1117-33, U4 MAX485E, U5 SN65HVD232, U6 ESP-01, Y1 12MHz, Y2 32.768kHz

Commit message: CPU Update Finish CPU V2 Design and finish CPU PiggyBack Board
Parts:
- removed J1: Micro_SD_Card, symbol Connector:Micro_SD_Card
- removed J3: USB_B_Micro, symbol Connector:USB_B_Micro
- added C35: 1µ, Capacitor_SMD:C_0805_2012Metric, symbol Device:C
- added J1: GSD09002SEU, eigene:GSD09002SEU, symbol Private_Lib:SD_Card
- added J3: USB_B, Connector_USB:USB_B_Lumberg_2411_02_Horizontal, symbol Connector:USB_B
- added J8: I2C, Connector_PinHeader_2.54mm:PinHeader_1x04_P2.54mm_Vertical, symbol Connector_Generic:Conn_01x04
- added Q7, Q8: BSS138, Package_TO_SOT_SMD:SOT-23, symbol Transistor_FET:BSS138
- added R12, R13: 10k, Resistor_SMD:R_0805_2012Metric, symbol Device:R
- added R47, R48, R49, R50: 4k7, Resistor_SMD:R_0805_2012Metric, symbol Device:R
- renumbered R12 to R14, R13 to R15, R14 to R16, R15 to R17, R16 to R18, R17 to R19, R18 to R20, R20 to R21, R21 to R22, R22 to R23, R19 to R24, R24 to R25, R23 to R26, R25 to R27, R26 to R28, R27 to R29, R28 to R30, R29 to R31, R30 to R32, R31 to R33, R32 to R34, R33 to R35, R34 to R36, R35 to R37, R36 to R38, R37 to R39, R38 to R40, R39 to R41, R40 to R42, R41 to R43, R42 to R44, R43 to R45, R44 to R46
Connections:
- net VCC is gone; now on net +5V: J5.1 (Pin_1), J5.2 (Pin_2), J5.3 (Pin_3), J5.4 (Pin_4)
- net +3V3: now also J1.4 (VDD), Q7.1 (G), Q8.1 (G), R12.1, R13.1, R47.2, R49.2
- net +5V: now also C35.1, J8.2 (Pin_2), R48.2, R50.2
- net GND: now also C35.2, J1.11 (SHELL2), J1.12 (SHELL1), J1.3 (VSS), J1.6 (VSS), J3.4 (GND), J3.5 (Shield), J8.1 (Pin_1)
- net LED_BOOT: now also U1.53 (PC12); no longer U1.59 (PB7)
- net LED_HEARTBEAT: now also U1.54 (PD2); no longer U1.58 (PB6)
- net SDIO_CardDetect: now reaches U1.20 (PA4)
- net SDIO_CardDetect: now also J1.10 (CARD_DETECT), R12.2
- net SDIO_WriteProtect: now reaches U1.21 (PA5)
- net SDIO_WriteProtect: now also J1.15 (Write_Protect), R13.2
- net D+: now reaches D7.1 (A1), R35.1
- net D+: now also J3.3 (D+)
- net at R16.2: now also J1.2 (CMD)
- net at R26.2: now also J1.8 (DAT1)
- net D-: now reaches D7.2 (A2), R36.1
- net D-: now also J3.2 (D-)
- net at R14.2: now also J1.9 (DAT2)
- net at R15.2: now also J1.1 (CD/DAT3)
- net at R20.2: now also J1.5 (CLK)
- net at R24.2: now also J1.7 (DAT0)
- net at FB1.1: now also J3.1 (VBUS)
- net USB_DM- renamed USB-
- net USB_DP+ renamed USB+
- new net I2C1_SCL: Q7.2 (S), R47.1, U1.58 (PB6)
- new net I2C1_SDA: Q8.2 (S), R49.1, U1.59 (PB7)
- new net SCL: J8.4 (Pin_4), Q7.3 (D), R48.1
- new net SDA: J8.3 (Pin_3), Q8.3 (D), R50.1
- no-connect marks 21 -> 16
Other:
- note added: "Grove-Port compatible"
- note added: "I2C"
- note added: "STM32 Peripherals ------------------- CAN1 = CAN @ 1Mbit/s USART1 = RS485 @ 1MBaud USART2 = ESP @ 250kBaud SPI2 = Reserved I2C1 = Reserved for PiggyBack SDIO = SD Card Interface USB_OTG_FS = Virtual Com Port"
- note removed: "STM32 Peripherals ------------------- CAN1 = CAN @ 1Mbit/s USART1 = RS485 @ 1MBaud USART2 = ESP @ 250kBaud SPI2 = Reserved SDIO = SD Card Interface USB_OTG_FS = Virtual Com Port"
- moved on the sheet: C1, C15, C16, C17, C18, C19, C2, C20, D3, D6, Q2, Q6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
