File: hardware/pcbs/CPU_V2/CPU_V2/CPU_V2.kicad_pcb (KiCad board)
At the start: 4 copper layers, 100 x 77 mm, 130 parts, among them J1 GSD09002SEU, J2 SWD, J3 USB_B, J4 24V_In, J5 Conn_02x05_Odd_Even, J6 Conn_02x03_Odd_Even, J7 SPI Conn, J8 I2C, Q1 BSS138, Q2 BSS138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

Commit message: CPU V2 Review
Parts:
- added ?: , eigene:ladder_4, F.Cu at (84.0, 142.1)
- added G***: LOGO, TheBrutzlers_Lib:approved_theBrutzler, F.Cu at (97.5, 100.0)
- moved JP1 1.64 mm to (170.1, 120.3)
- moved C29 1.26 mm to (166.5, 70.7), turned to 180 degrees
- moved FB1 0.26 mm to (166.4, 126.5)
Routing:
- net GND: track 174.5 -> 194.4 mm, vias 129 -> 124
- net /VBAT: track 40.8 -> 39.6 mm
- net Net-(C14-Pad2): track 12.8 -> 14.0 mm
- net /BUS+: track 10.0 -> 9.16 mm
- net +3V3: track 97.3 -> 96.4 mm
- net Net-(C10-Pad1): track 9.19 -> 10.0 mm
- net +5V: track 128.5 -> 127.7 mm
- added copper zone on F.Cu, net +3V3
