File: hardware/pcbs/CPU_V2/CPU_V2/CPU_V2.kicad_sch (KiCad schematic)
At the start: 127 parts, among them J1 GSD09002SEU, J2 SWD, J3 USB_B, J4 24V_In, J5 Conn_02x05_Odd_Even, J6 Conn_02x03_Odd_Even, J7 SPI Conn, J8 I2C, Q1 BSS138, Q2 BSS138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

Commit message: CPU V2 Review
Changed lines of the file:
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@@
       (effects (font (size 1.27 1.27)) hide)
     )
-    (property "Datasheet" "~" (id 3) (at 177.8 270.51 0)
+    (property "Datasheet" "https://www.mouser.de/datasheet/2/54/cdsot23-t24can-q-1534349.pdf" (id 3) (at 177.8 270.51 0)
       (effects (font (size 1.27 1.27)) hide)
     )
@@
   (symbol (lib_id "Device:D_TVS_Dual_AAC") (at 368.3 124.46 0) (mirror y) (unit 1)
     (in_bom yes) (on_board yes) (fields_autoplaced)
-    (property "Reference" "D7" (id 0) (at 368.3 119.4902 0))
-    (property "Value" "CDSOT23-T24-Q" (id 1) (at 368.3 122.0271 0))
+    (property "Reference" "D7" (id 0) (at 368.3 118.11 0))
+    (property "Value" "CDSOT23-T24-Q" (id 1) (at 368.3 120.65 0))
     (property "Footprint" "Package_TO_SOT_SMD:SOT-23" (id 2) (at 372.11 124.46 0)
       (effects (font (size 1.27 1.27)) hide)
     )
-    (property "Datasheet" "~" (id 3) (at 372.11 124.46 0)
-      (effects (font (size 1.27 1.27)) hide)
-    )
+    (property "Datasheet" "https://www.mouser.de/datasheet/2/54/cdsot23-t24can-q-1534349.pdf" (id 3) (at 372.11 124.46 0)
+      (effects (font (size 1.27 1.27)) hide)
+    )
