File: hardware/pcbs/CPU_V2/CPU_PiggyBack/CPU_PiggyBack.kicad_pcb (KiCad board)
At the start: 4 copper layers, 100 x 77 mm, 142 parts, among them J1 I2C, J2 TBL009-500-02GY-2GY, J3 TBL009-500-02GY-2GY, J4 TBL009-500-02GY-2GY, J5 TBL009-500-02GY-2GY, J6 TBL009-500-02GY-2GY, Q1 BCX53, Q10 BC856, Q11 BC856, Q12 BC856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

Commit message: case design for new CPU with piggyback
Parts:
- moved R45 1.91 mm to (178.2, 72.6)
- moved R46 1.91 mm to (178.2, 76.8)
- moved R47 1.91 mm to (178.2, 81.0)
- moved R48 1.91 mm to (178.2, 85.2)
- moved R53 1.91 mm to (178.2, 89.4)
- moved R54 1.91 mm to (178.2, 93.6)
- moved R55 1.91 mm to (178.2, 97.8)
- moved R56 1.91 mm to (178.2, 102.0)
- moved D22 1.91 mm to (184.2, 72.6)
- moved D23 1.91 mm to (184.2, 76.8)
- moved D24 1.91 mm to (184.2, 81.0)
- moved D25 1.91 mm to (184.2, 85.2)
- moved D26 1.91 mm to (184.2, 89.4)
- moved D27 1.91 mm to (184.2, 93.6)
- moved D28 1.91 mm to (184.2, 97.8)
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Routing:
- net OUT_3: track 74.0 -> 72.1 mm
- net OUT_2: track 80.2 -> 78.3 mm
- net OUT_1: track 86.4 -> 84.5 mm
- net OUT_0: track 93.4 -> 91.5 mm
- net IN_2: track 44.0 -> 42.1 mm
- net IN_1: track 53.6 -> 51.7 mm
- net IN_0: track 58.2 -> 56.3 mm
- net IN_3: track 41.9 -> 40.0 mm
Other:
- board text added: "SynPLC DIO4/4 Rev 1.0"
- board text added: "https://github.com/Synthron/SynPLC"
- board text removed: "SynPLC DIO4/4 Rev 1"

Commit message: CPU V2 Review
Parts:
- added ?: , eigene:ladder_4, F.Cu at (102.5, 122.9)
- added D30: 6v8, Diode_SMD:D_MiniMELF, F.Cu at (104.2, 81.4)
- added D31: 6v8, Diode_SMD:D_MiniMELF, F.Cu at (106.7, 81.4)
- added D32: 6v8, Diode_SMD:D_MiniMELF, F.Cu at (109.2, 81.4)
- added D33: 6v8, Diode_SMD:D_MiniMELF, F.Cu at (111.8, 81.4)
- added G***: LOGO, TheBrutzlers_Lib:approved_theBrutzler, F.Cu at (176.2, 115.2)
- added R57: 10k, Resistor_SMD:R_0805_2012Metric, F.Cu at (121.8, 85.7)
- added R58: 10k, Resistor_SMD:R_0805_2012Metric, F.Cu at (119.3, 85.7)
- added R59: 10k, Resistor_SMD:R_0805_2012Metric, F.Cu at (124.3, 85.7)
- added R60: 10k, Resistor_SMD:R_0805_2012Metric, F.Cu at (126.9, 85.7)
Connections:
- F1 pad 1: Net-(F1-Pad1) -> Net-(D30-Pad1)
- F2 pad 1: Net-(F2-Pad1) -> Net-(D31-Pad1)
- F3 pad 1: Net-(F3-Pad1) -> Net-(D32-Pad1)
- F4 pad 1: Net-(F4-Pad1) -> Net-(D33-Pad1)
- FB3 pad 2: Net-(F1-Pad1) -> Net-(D30-Pad1)
- FB4 pad 2: Net-(F2-Pad1) -> Net-(D31-Pad1)
- FB5 pad 2: Net-(F3-Pad1) -> Net-(D32-Pad1)
- FB6 pad 2: Net-(F4-Pad1) -> Net-(D33-Pad1)
- R10 pad 1: Net-(F2-Pad1) -> Net-(D31-Pad2)
- R12 pad 2: Net-(F2-Pad1) -> Net-(D31-Pad1)
- R13 pad 1: Net-(F3-Pad1) -> Net-(D32-Pad2)
- R16 pad 2: Net-(F3-Pad1) -> Net-(D32-Pad1)
- R17 pad 1: Net-(F4-Pad1) -> Net-(D33-Pad2)
- R20 pad 2: Net-(F4-Pad1) -> Net-(D33-Pad1)
- R6 pad 1: Net-(F1-Pad1) -> Net-(D30-Pad2)
- R8 pad 2: Net-(F1-Pad1) -> Net-(D30-Pad1)
- U3 pad 10: Net-(Q4-Pad1) -> Net-(R60-Pad1)
- U3 pad 12: Net-(Q3-Pad1) -> Net-(R59-Pad1)
- U3 pad 14: Net-(Q2-Pad1) -> Net-(R57-Pad1)
- U3 pad 16: Net-(Q1-Pad1) -> Net-(R58-Pad1)
Routing:
- net Net-(F4-Pad1): track 45.6 -> 0.00 mm, vias 2 -> 0
- net Net-(F3-Pad1): track 40.9 -> 0.00 mm, vias 2 -> 0
- net Net-(D33-Pad1): track 0.00 -> 37.3 mm, vias 0 -> 2
- net Net-(F2-Pad1): track 35.9 -> 0.00 mm, vias 2 -> 0
- net Net-(D32-Pad1): track 0.00 -> 32.2 mm, vias 0 -> 2
- net Net-(F1-Pad1): track 30.6 -> 0.00 mm, vias 2 -> 0
- net Net-(D30-Pad1): track 0.00 -> 29.5 mm, vias 0 -> 2
- net Net-(D31-Pad1): track 0.00 -> 28.5 mm, vias 0 -> 2
- net Net-(Q1-Pad1): track 34.9 -> 30.4 mm
- net Net-(Q2-Pad1): track 29.6 -> 25.2 mm
- net Net-(Q3-Pad1): track 24.1 -> 19.7 mm
- net Net-(Q4-Pad1): track 22.0 -> 17.6 mm
- net Net-(R57-Pad1): track 0.00 -> 2.70 mm
- net Net-(R60-Pad1): track 0.00 -> 2.70 mm
- net Net-(R59-Pad1): track 0.00 -> 2.70 mm
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- added copper zone on F.Cu, net Net-(D1-Pad1)
- added copper zone on F.Cu, net Net-(D1-Pad2)

Commit message: update
Parts:
- R11, R15, R19, R7: value 10k -> 100k
Changed lines of the file:
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@@
       (effects (font (size 0.6 0.6) (thickness 0.1)))
     )
-    (fp_text value "10k" (at 0 1.65 90) (layer "F.Fab")
+    (fp_text value "100k" (at 0 1.65 90) (layer "F.Fab")
       (effects (font (size 1 1) (thickness 0.15)))
     )
@@
       (effects (font (size 0.6 0.6) (thickness 0.1)))
     )
-    (fp_text value "10k" (at 0 1.65 90) (layer "F.Fab")
+    (fp_text value "100k" (at 0 1.65 90) (layer "F.Fab")
       (effects (font (size 1 1) (thickness 0.15)))
     )
@@
       (effects (font (size 0.6 0.6) (thickness 0.1)))
     )
-    (fp_text value "10k" (at 0 1.65 90) (layer "F.Fab")
+    (fp_text value "100k" (at 0 1.65 90) (layer "F.Fab")
       (effects (font (size 1 1) (thickness 0.15)))
     )
@@
       (effects (font (size 0.6 0.6) (thickness 0.1)))
     )
-    (fp_text value "10k" (at 0 1.65 90) (layer "F.Fab")
+    (fp_text value "100k" (at 0 1.65 90) (layer "F.Fab")
       (effects (font (size 1 1) (thickness 0.15)))
     )
