File: hardware/pcbs/CPU_V2/CPU_PiggyBack/CPU_PiggyBack.kicad_sch (KiCad schematic)
At the start: 139 parts, among them J1 I2C, J2 TBL009-500-02GY-2GY, J3 TBL009-500-02GY-2GY, J4 TBL009-500-02GY-2GY, J5 TBL009-500-02GY-2GY, J6 TBL009-500-02GY-2GY, Q1 BCX53, Q10 BC856, Q11 BC856, Q12 BC856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

Commit message: CPU V2 Review
Parts:
- added D30, D31, D32, D33: 6v8, Diode_SMD:D_MiniMELF, symbol Device:D_Zener
- added R57, R58, R59, R60: 10k, Resistor_SMD:R_0805_2012Metric, symbol Device:R
Connections:
- net at F4.1, FB6.2, R20.2: now also D33.1 (K); no longer R17.1
- net at Q2.1 (B), R11.1: now also R57.2; no longer U3.14
- net at F1.1, FB3.2, R8.2: now also D30.1 (K); no longer R6.1
- net at Q4.1 (B), R19.1: now also R60.2; no longer U3.10
- net at F3.1, FB5.2, R16.2: now also D32.1 (K); no longer R13.1
- net at Q1.1 (B), R7.1: now also R58.2; no longer U3.16
- net at Q3.1 (B), R15.1: now also R59.2; no longer U3.12
- net at F2.1, FB4.2, R12.2: now also D31.1 (K); no longer R10.1
- new net: R57.1, U3.14
- new net: R59.1, U3.12
- new net: D32.2 (A), R13.1
- new net: R58.1, U3.16
- new net: R60.1, U3.10
- new net: D33.2 (A), R17.1
- new net: D30.2 (A), R6.1
- new net: D31.2 (A), R10.1

Commit message: update
Parts:
- R11, R15, R19, R7: value 10k -> 100k
Changed lines of the file:
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@@
       (effects (font (size 1.27 1.27)) (justify right))
     )
-    (property "Value" "10k" (id 1) (at 127.508 110.363 0)
+    (property "Value" "100k" (id 1) (at 127.508 110.363 0)
       (effects (font (size 1.27 1.27)) (justify right))
     )
@@
       (effects (font (size 1.27 1.27)) (justify right))
     )
-    (property "Value" "10k" (id 1) (at 127.508 49.403 0)
+    (property "Value" "100k" (id 1) (at 127.508 49.403 0)
       (effects (font (size 1.27 1.27)) (justify right))
     )
@@
       (effects (font (size 1.27 1.27)) (justify right))
     )
-    (property "Value" "10k" (id 1) (at 127.508 90.043 0)
+    (property "Value" "100k" (id 1) (at 127.508 90.043 0)
       (effects (font (size 1.27 1.27)) (justify right))
     )
@@
       (effects (font (size 1.27 1.27)) (justify right))
     )
-    (property "Value" "10k" (id 1) (at 127.508 69.723 0)
+    (property "Value" "100k" (id 1) (at 127.508 69.723 0)
       (effects (font (size 1.27 1.27)) (justify right))
     )
@@
     )
     (path "/ded0eb64-6f74-4ae7-9c6f-2e98a7ee83ca"
-      (reference "R7") (unit 1) (value "10k") (footprint "Resistor_SMD:R_0805_2012Metric")
+      (reference "R7") (unit 1) (value "100k") (footprint "Resistor_SMD:R_0805_2012Metric")
     )
     (path "/3f046322-eaee-407d-9c92-080966663a70"
@@
     )
     (path "/efd97b96-4170-4f0a-832b-a4e20040128e"
-      (reference "R11") (unit 1) (value "10k") (footprint "Resistor_SMD:R_0805_2012Metric")
+      (reference "R11") (unit 1) (value "100k") (footprint "Resistor_SMD:R_0805_2012Metric")
     )
     (path "/7362028c-bb37-4b22-984d-a9b98eaf7fe2"
@@
     )
     (path "/dff80299-42dc-428e-8ff9-5b5bda3de7aa"
-      (reference "R15") (unit 1) (value "10k") (footprint "Resistor_SMD:R_0805_2012Metric")
+      (reference "R15") (unit 1) (value "100k") (footprint "Resistor_SMD:R_0805_2012Metric")
     )
     (path "/a57363f1-5fbf-4fc4-94a2-80f0a6d72db2"
@@
     )
     (path "/281ae7e8-07b8-4bd3-901a-76dba923f70c"
-      (reference "R19") (unit 1) (value "10k") (footprint "Resistor_SMD:R_0805_2012Metric")
+      (reference "R19") (unit 1) (value "100k") (footprint "Resistor_SMD:R_0805_2012Metric")
     )
     (path "/6885f791-228d-4992-be7d-4a2d8d9ca9e6"
